File: bitaxe.kicad_sch (KiCad schematic)
At the start: 101 parts, among them IC1 BM1387, IC2 BM1387, IC3 TCR2EF18, IC4 TCR2EF18, J1 Conn_01x01, J2 Conn_01x01, J3 Conn_01x05, J4 Conn_01x02, J5 Conn_01x03, Y1 25MHz

Commit message: flipped (again) C17 and C18 for #1
Parts:
- C17, C18: footprint Capacitor_Tantalum_SMD:CP_EIA-7343-31_Kemet-D_Pad2.25x2.55mm_HandSolder_flip -> Capacitor_Tantalum_SMD:CP_EIA-7343-31_Kemet-D_Pad2.25x2.55mm_HandSolder
Changed lines of the file:
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@@
       (effects (font (size 1.27 1.27)) (justify left))
     )
-    (property "Footprint" "Capacitor_Tantalum_SMD:CP_EIA-7343-31_Kemet-D_Pad2.25x2.55mm_HandSolder_flip" (id 2) (at 235.9152 70.485 0)
+    (property "Footprint" "Capacitor_Tantalum_SMD:CP_EIA-7343-31_Kemet-D_Pad2.25x2.55mm_HandSolder" (id 2) (at 235.9152 70.485 0)
       (effects (font (size 1.27 1.27)) hide)
     )
@@
       (effects (font (size 1.27 1.27)) (justify left))
     )
-    (property "Footprint" "Capacitor_Tantalum_SMD:CP_EIA-7343-31_Kemet-D_Pad2.25x2.55mm_HandSolder_flip" (id 2) (at 234.6452 149.225 0)
+    (property "Footprint" "Capacitor_Tantalum_SMD:CP_EIA-7343-31_Kemet-D_Pad2.25x2.55mm_HandSolder" (id 2) (at 234.6452 149.225 0)
       (effects (font (size 1.27 1.27)) hide)
     )
@@
     )
     (path "/acfd78ad-ef0a-414c-9378-060e937bcb37"
-      (reference "C17") (unit 1) (value "330uF") (footprint "Capacitor_Tantalum_SMD:CP_EIA-7343-31_Kemet-D_Pad2.25x2.55mm_HandSolder_flip")
+      (reference "C17") (unit 1) (value "330uF") (footprint "Capacitor_Tantalum_SMD:CP_EIA-7343-31_Kemet-D_Pad2.25x2.55mm_HandSolder")
     )
     (path "/358da881-61fd-4ea9-810a-034bc845f90c"
-      (reference "C18") (unit 1) (value "330uF") (footprint "Capacitor_Tantalum_SMD:CP_EIA-7343-31_Kemet-D_Pad2.25x2.55mm_HandSolder_flip")
+      (reference "C18") (unit 1) (value "330uF") (footprint "Capacitor_Tantalum_SMD:CP_EIA-7343-31_Kemet-D_Pad2.25x2.55mm_HandSolder")
     )
     (path "/9e197296-7ecf-47fb-b06b-346b771006ce"
       (reference "C19") (unit 1) (value "0.1uF") (footprint "DayMiner:C0402")
     )
-    (path "/82494300-14ee-4d15-aa1d-70b7cbf70aba"
+    (path "/82494300-14ee-4d15-aa1d-70b7cbf70abb"
       (reference "C20") (unit 1) (value "0.1uF") (footprint "DayMiner:C0402")
     )
