File: bitaxeHex.kicad_pcb (KiCad board)
At the start: 4 copper layers, 56.5 x 99.8 mm, 153 parts, among them IC1 BM1397_mode1, J1 Conn_01x01, J10 FTSH-105-01-F-DV-K_SAI, J2 Conn_01x01, J3 Conn_01x05, J4 Conn_01x04, J5 TC2030-IDC, J6 Conn_01x08, J7 Conn_01x02, J9 Conn_01x04, Q1 CSD17311Q5, Q2 CSD17311Q5, U1 25MHz, U10 DS4432U+, U11 RT9080-33GJ5, U12 ESP32-S3-WROOM-1, U13 CLX6E-FKC, U2 TXB0104RGYR, U3 SN74AXC1T45DBVR, U4 CLX6E-FKC, U5 MCP1824, U6 MCP1824, U7 EMC2101, U8 INA260, U9 TPS40305, Y1 32.768kHz

Commit message: fixed the floating gnd net issue. started placement
Parts:
- removed J10: FTSH-105-01-F-DV-K_SAI, bitaxe:FTSH-105-01-F-DV-K
- removed J3: Conn_01x05, Connector_PinHeader_2.54mm:PinHeader_1x05_P2.54mm_Vertical
- removed J9: Conn_01x04, Connector_PinHeader_2.54mm:PinHeader_1x04_P2.54mm_Vertical
- removed JP1, JP2: SolderJumper_2_Open, Jumper:SolderJumper-2_P1.3mm_Open_RoundedPad1.0x1.5mm
- removed JP3: SolderJumper_2_Bridged, Jumper:SolderJumper-2_P1.3mm_Bridged2Bar_RoundedPad1.0x1.5mm
- removed JP4: JTAG Source, Jumper:SolderJumper-3_P1.3mm_Bridged2Bar12_Pad1.0x1.5mm
- removed TP29, TP30, TP31, TP32: TestPoint, TestPoint:TestPoint_Pad_D1.5mm
- removed kibuzzard-6387EEBE: G***, kibuzzard-6387EEBE
- removed kibuzzard-6387EECB: G***, kibuzzard-6387EECB
- removed kibuzzard-6392B1E5: G***, kibuzzard-6392B1E5
- removed kibuzzard-63D74789: G***, kibuzzard-63D74789
- added C100: 587-5514-1-ND, Capacitor_SMD:C_0402_1005Metric, F.Cu at (-45.9, 186.9)
- added C101: 311-3342-1-ND, Capacitor_SMD:C_0402_1005Metric, F.Cu at (-43.0, 171.2)
- added C102: 587-5514-1-ND, Capacitor_SMD:C_0402_1005Metric, F.Cu at (-43.0, 173.1)
- added C103: 587-5514-1-ND, Capacitor_SMD:C_0402_1005Metric, F.Cu at (-43.0, 175.1)
- added C104: 587-5514-1-ND, Capacitor_SMD:C_0402_1005Metric, F.Cu at (-43.0, 177.1)
- added C105: 330uF, Capacitor_Tantalum_SMD:CP_EIA-7343-31_Kemet-D_Pad2.25x2.55mm_HandSolder, F.Cu at (-47.9, 196.7)
- added C106: 587-5514-1-ND, Capacitor_SMD:C_0402_1005Metric, F.Cu at (-43.0, 179.1)
- added C107: 587-5514-1-ND, Capacitor_SMD:C_0402_1005Metric, F.Cu at (-43.0, 181.0)
- added C108: 587-5514-1-ND, Capacitor_SMD:C_0402_1005Metric, F.Cu at (-43.0, 183.0)
- added C109: 587-5514-1-ND, Capacitor_SMD:C_0402_1005Metric, F.Cu at (-43.0, 185.0)
- added C110: 587-5514-1-ND, Capacitor_SMD:C_0402_1005Metric, F.Cu at (-43.0, 186.9)
- added C111: 587-5514-1-ND, Capacitor_SMD:C_0402_1005Metric, F.Cu at (-35.2, 171.2)
- added C112: 587-5514-1-ND, Capacitor_SMD:C_0402_1005Metric, F.Cu at (-35.2, 173.1)
- added C113: 587-5514-1-ND, Capacitor_SMD:C_0402_1005Metric, F.Cu at (-35.2, 175.1)
- added C114: 587-5514-1-ND, Capacitor_SMD:C_0402_1005Metric, F.Cu at (-35.2, 177.1)
- added C115: 587-5514-1-ND, Capacitor_SMD:C_0402_1005Metric, F.Cu at (-35.2, 179.1)
- added C116: 311-3342-1-ND, Capacitor_SMD:C_0402_1005Metric, F.Cu at (-35.2, 181.0)
- added C117: 311-3342-1-ND, Capacitor_SMD:C_0402_1005Metric, F.Cu at (-35.2, 183.0)
- added C118: 311-3342-1-ND, Capacitor_SMD:C_0402_1005Metric, F.Cu at (-35.2, 185.0)
- added C119: 587-5514-1-ND, Capacitor_SMD:C_0402_1005Metric, F.Cu at (-35.2, 186.9)
- added C120: 311-3342-1-ND, Capacitor_SMD:C_0402_1005Metric, F.Cu at (-32.4, 171.2)
- added C121: 587-5514-1-ND, Capacitor_SMD:C_0402_1005Metric, F.Cu at (-32.4, 173.1)
- added C122: 587-5514-1-ND, Capacitor_SMD:C_0402_1005Metric, F.Cu at (-32.4, 175.1)
- added C123: 1uF, Capacitor_SMD:C_0402_1005Metric, F.Cu at (-32.4, 177.1)
- added C124: 1uF, Capacitor_SMD:C_0402_1005Metric, F.Cu at (-32.4, 179.1)
- added C125: 587-5514-1-ND, Capacitor_SMD:C_0402_1005Metric, F.Cu at (-32.4, 181.0)
- added C126: 330uF, Capacitor_Tantalum_SMD:CP_EIA-7343-31_Kemet-D_Pad2.25x2.55mm_HandSolder, F.Cu at (-31.5, 190.8)
- added C127: 587-5514-1-ND, Capacitor_SMD:C_0402_1005Metric, F.Cu at (-32.4, 183.0)
- added C128: 587-5514-1-ND, Capacitor_SMD:C_0402_1005Metric, F.Cu at (-32.4, 185.0)
- added C129: 587-5514-1-ND, Capacitor_SMD:C_0402_1005Metric, F.Cu at (-32.4, 186.9)
- added C130: 587-5514-1-ND, Capacitor_SMD:C_0402_1005Metric, F.Cu at (-29.5, 171.2)
- added C131: 587-5514-1-ND, Capacitor_SMD:C_0402_1005Metric, F.Cu at (-29.5, 173.1)
- added C132: 587-5514-1-ND, Capacitor_SMD:C_0402_1005Metric, F.Cu at (-29.5, 175.1)
- added C133: 587-5514-1-ND, Capacitor_SMD:C_0402_1005Metric, F.Cu at (-29.5, 177.1)
- added C134: 587-5514-1-ND, Capacitor_SMD:C_0402_1005Metric, F.Cu at (-29.5, 179.1)
- added C135: 587-5514-1-ND, Capacitor_SMD:C_0402_1005Metric, F.Cu at (-29.5, 181.0)
- added C136: 587-5514-1-ND, Capacitor_SMD:C_0402_1005Metric, F.Cu at (-29.5, 183.0)
- added C137: 311-3342-1-ND, Capacitor_SMD:C_0402_1005Metric, F.Cu at (-29.5, 185.0)
- added C138: 587-5514-1-ND, Capacitor_SMD:C_0402_1005Metric, F.Cu at (-29.5, 186.9)
- added C139: 311-3342-1-ND, Capacitor_SMD:C_0402_1005Metric, F.Cu at (-26.6, 171.2)
- added C140: 587-5514-1-ND, Capacitor_SMD:C_0402_1005Metric, F.Cu at (-26.6, 173.1)
- added C141: 587-5514-1-ND, Capacitor_SMD:C_0402_1005Metric, F.Cu at (-26.6, 175.1)
- added C142: 587-5514-1-ND, Capacitor_SMD:C_0402_1005Metric, F.Cu at (-26.6, 177.1)
- added C143: 330uF, Capacitor_Tantalum_SMD:CP_EIA-7343-31_Kemet-D_Pad2.25x2.55mm_HandSolder, F.Cu at (-31.5, 196.7)
- added C144: 587-5514-1-ND, Capacitor_SMD:C_0402_1005Metric, F.Cu at (-26.6, 179.1)
- added C145: 587-5514-1-ND, Capacitor_SMD:C_0402_1005Metric, F.Cu at (-26.6, 181.0)
- added C146: 587-5514-1-ND, Capacitor_SMD:C_0402_1005Metric, F.Cu at (-26.6, 183.0)
- added C147: 587-5514-1-ND, Capacitor_SMD:C_0402_1005Metric, F.Cu at (-26.6, 185.0)
- added C148: 587-5514-1-ND, Capacitor_SMD:C_0402_1005Metric, F.Cu at (-26.6, 186.9)
- added C48: 587-5514-1-ND, Capacitor_SMD:C_0402_1005Metric, F.Cu at (-51.6, 208.5)
- added C53: 311-3342-1-ND, Capacitor_SMD:C_0402_1005Metric, F.Cu at (-51.6, 210.4)
- added C54: 587-5514-1-ND, Capacitor_SMD:C_0402_1005Metric, F.Cu at (-51.6, 212.4)
- added C55: 311-3342-1-ND, Capacitor_SMD:C_0402_1005Metric, F.Cu at (-51.6, 214.4)
- added C56: 587-5514-1-ND, Capacitor_SMD:C_0402_1005Metric, F.Cu at (-48.8, 208.5)
- added C57: 587-5514-1-ND, Capacitor_SMD:C_0402_1005Metric, F.Cu at (-48.8, 210.4)
- added C58: 587-5514-1-ND, Capacitor_SMD:C_0402_1005Metric, F.Cu at (-48.8, 212.4)
- added C59: 330uF, Capacitor_Tantalum_SMD:CP_EIA-7343-31_Kemet-D_Pad2.25x2.55mm_HandSolder, F.Cu at (-58.1, 204.5)
- added C60: 587-5514-1-ND, Capacitor_SMD:C_0402_1005Metric, F.Cu at (-48.8, 214.4)
- added C61: 587-5514-1-ND, Capacitor_SMD:C_0402_1005Metric, F.Cu at (-45.9, 208.5)
- added C62: 587-5514-1-ND, Capacitor_SMD:C_0402_1005Metric, F.Cu at (-45.9, 210.4)
- added C63: 587-5514-1-ND, Capacitor_SMD:C_0402_1005Metric, F.Cu at (-45.9, 212.4)
- added C64: 587-5514-1-ND, Capacitor_SMD:C_0402_1005Metric, F.Cu at (-45.9, 214.4)
- added C65: 470pF, Capacitor_SMD:C_0402_1005Metric, F.Cu at (-30.6, 202.6)
- added C66: 470pF, Capacitor_SMD:C_0402_1005Metric, F.Cu at (-30.6, 204.6)
- added C67: 311-3342-1-ND, Capacitor_SMD:C_0402_1005Metric, F.Cu at (-30.6, 206.5)
- added C68: 311-3342-1-ND, Capacitor_SMD:C_0402_1005Metric, F.Cu at (-30.6, 208.5)
- added C69: 220uF, Capacitor_SMD:CP_Elec_6.3x7.7, F.Cu at (-37.2, 205.7)
- added C70: 220uF, Capacitor_SMD:CP_Elec_6.3x7.7, F.Cu at (-37.2, 213.8)
- added C71: 311-3342-1-ND, Capacitor_SMD:C_0402_1005Metric, F.Cu at (-30.6, 210.5)
- added C72: 311-3342-1-ND, Capacitor_SMD:C_0402_1005Metric, F.Cu at (-30.6, 212.5)
- added C73: 587-5514-1-ND, Capacitor_SMD:C_0402_1005Metric, F.Cu at (-51.6, 171.2)
- added C74: 587-5514-1-ND, Capacitor_SMD:C_0402_1005Metric, F.Cu at (-51.6, 173.1)
- added C75: 587-5514-1-ND, Capacitor_SMD:C_0402_1005Metric, F.Cu at (-51.6, 175.1)
- added C76: 587-5514-1-ND, Capacitor_SMD:C_0402_1005Metric, F.Cu at (-51.6, 177.1)
- added C77: 587-5514-1-ND, Capacitor_SMD:C_0402_1005Metric, F.Cu at (-51.6, 179.1)
- added C78: 311-3342-1-ND, Capacitor_SMD:C_0402_1005Metric, F.Cu at (-51.6, 181.0)
- added C79: 311-3342-1-ND, Capacitor_SMD:C_0402_1005Metric, F.Cu at (-51.6, 183.0)
- added C80: 311-3342-1-ND, Capacitor_SMD:C_0402_1005Metric, F.Cu at (-51.6, 185.0)
- added C81: 587-5514-1-ND, Capacitor_SMD:C_0402_1005Metric, F.Cu at (-51.6, 186.9)
- added C82: 311-3342-1-ND, Capacitor_SMD:C_0402_1005Metric, F.Cu at (-48.8, 171.2)
- added C83: 587-5514-1-ND, Capacitor_SMD:C_0402_1005Metric, F.Cu at (-48.8, 173.1)
- added C84: 587-5514-1-ND, Capacitor_SMD:C_0402_1005Metric, F.Cu at (-48.8, 175.1)
- added C85: 1uF, Capacitor_SMD:C_0402_1005Metric, F.Cu at (-48.8, 177.1)
- added C86: 1uF, Capacitor_SMD:C_0402_1005Metric, F.Cu at (-48.8, 179.1)
- added C87: 587-5514-1-ND, Capacitor_SMD:C_0402_1005Metric, F.Cu at (-48.8, 181.0)
- added C88: 330uF, Capacitor_Tantalum_SMD:CP_EIA-7343-31_Kemet-D_Pad2.25x2.55mm_HandSolder, F.Cu at (-47.9, 190.8)
- added C89: 587-5514-1-ND, Capacitor_SMD:C_0402_1005Metric, F.Cu at (-48.8, 183.0)
- added C90: 587-5514-1-ND, Capacitor_SMD:C_0402_1005Metric, F.Cu at (-48.8, 185.0)
- added C91: 587-5514-1-ND, Capacitor_SMD:C_0402_1005Metric, F.Cu at (-48.8, 186.9)
- added C92: 587-5514-1-ND, Capacitor_SMD:C_0402_1005Metric, F.Cu at (-45.9, 171.2)
- added C93: 587-5514-1-ND, Capacitor_SMD:C_0402_1005Metric, F.Cu at (-45.9, 173.1)
- added C94: 587-5514-1-ND, Capacitor_SMD:C_0402_1005Metric, F.Cu at (-45.9, 175.1)
- added C95: 587-5514-1-ND, Capacitor_SMD:C_0402_1005Metric, F.Cu at (-45.9, 177.1)
- added C96: 587-5514-1-ND, Capacitor_SMD:C_0402_1005Metric, F.Cu at (-45.9, 179.1)
- added C97: 587-5514-1-ND, Capacitor_SMD:C_0402_1005Metric, F.Cu at (-45.9, 181.0)
- added C98: 587-5514-1-ND, Capacitor_SMD:C_0402_1005Metric, F.Cu at (-45.9, 183.0)
- added C99: 311-3342-1-ND, Capacitor_SMD:C_0402_1005Metric, F.Cu at (-45.9, 185.0)
- added D1: SS310_C85658, lcsc:SMA_L4.3-W2.6-LS5.2-RD, F.Cu at (-16.8, 211.2)
- added H10: MountingHole, MountingHole:MountingHole_3.5mm, F.Cu at (186.0, 119.4)
- added H7: MountingHole, MountingHole:MountingHole_3.5mm, F.Cu at (101.0, 78.0)
- added H8: MountingHole, MountingHole:MountingHole_3.5mm, F.Cu at (142.3, 119.5)
- added H9: MountingHole, MountingHole:MountingHole_3.5mm, F.Cu at (144.6, 78.0)
- added IC2: BM1397_mode1, bitaxe:BM1397, B.Cu at (87.9, 99.6)
- added IC3: BM1397_mode0, bitaxe:BM1397, B.Cu at (111.6, 99.4)
- added IC4: BM1397_mode0, bitaxe:BM1397, B.Cu at (132.2, 99.4)
- added IC5: BM1397_mode1, bitaxe:BM1397, B.Cu at (155.1, 99.6)
- added IC6: BM1397_mode1, bitaxe:BM1397, B.Cu at (175.9, 99.6)
- added Q3: NTMFS5C673NLT1G, bitaxe:NTMFS5C673NLT1G, F.Cu at (99.3, 57.1)
- added Q4: CSD17577Q5A, bitaxe:CSD17577Q5A, F.Cu at (78.9, 57.2)
- added R30: 5.6k, Resistor_SMD:R_0402_1005Metric, F.Cu at (-30.6, 214.4)
- added R31: 5.6k, Resistor_SMD:R_0402_1005Metric, F.Cu at (-30.6, 216.4)
- added R32: 0, Resistor_SMD:R_0402_1005Metric, F.Cu at (-40.1, 171.2)
- added R33: 0, Resistor_SMD:R_0402_1005Metric, F.Cu at (-40.1, 173.2)
- added R34: 0, Resistor_SMD:R_0402_1005Metric, F.Cu at (-40.1, 175.2)
- added R35: 1, Resistor_SMD:R_2512_6332Metric, F.Cu at (-58.9, 191.4)
- added R37: 0, Resistor_SMD:R_0402_1005Metric, F.Cu at (-40.1, 177.2)
- added R38: 0, Resistor_SMD:R_0402_1005Metric, F.Cu at (-40.1, 179.1)
- added R39: 0, Resistor_SMD:R_0402_1005Metric, F.Cu at (-40.1, 181.1)
- added R40: 0, Resistor_SMD:R_0402_1005Metric, F.Cu at (-13.6, 171.2)
- added R41: 0, Resistor_SMD:R_0402_1005Metric, F.Cu at (-13.6, 173.2)
- added R42: 0, Resistor_SMD:R_0402_1005Metric, F.Cu at (-13.6, 175.2)
- added R43: 1, Resistor_SMD:R_2512_6332Metric, F.Cu at (-20.9, 191.4)
- added R44: 1, Resistor_SMD:R_2512_6332Metric, F.Cu at (-20.9, 196.3)
- added R45: 0, Resistor_SMD:R_0402_1005Metric, F.Cu at (-13.6, 177.2)
- added R46: 0, Resistor_SMD:R_0402_1005Metric, F.Cu at (-13.6, 179.1)
- added R47: 0, Resistor_SMD:R_0402_1005Metric, F.Cu at (-13.6, 181.1)
- added SW1: GT-TC029B-H025-L1N, lcsc:SW-SMD_L3.9-W3.0-P4.45, F.Cu at (-23.8, 211.3)
- added SW2: GT-TC029B-H025-L1N, lcsc:SW-SMD_L3.9-W3.0-P4.45, F.Cu at (-23.8, 215.6)
- added TP20: TestPoint, TestPoint:TestPoint_Pad_D1.5mm, F.Cu at (-61.5, 195.6)
- added U14: MCP1824T-0802E, Package_TO_SOT_SMD:SOT-23-5, F.Cu at (-13.9, 191.2)
- added USB1: U254-051T-4BHJ25-F2S, lcsc:MICRO-USB-SMD_U254-051T-4BHJ25-F2S, F.Cu at (-22.2, 204.3)
- added X1: OT322525MJBA4SL, lcsc:OSC-SMD_4P-L3.2-W2.5-BL, F.Cu at (-50.1, 203.8)
- C1: value 311-3342-1-ND -> 22uF; footprint Capacitor_SMD:C_0402_1005Metric -> Capacitor_SMD:C_2220_5650Metric
- C10: value 587-5514-1-ND -> 0.33uF
- C11, C15, C16: value 587-5514-1-ND -> 1uF
- C12, C14: value 587-5514-1-ND -> 0.1uF
- C13: value 330uF -> 4.7uF; footprint Capacitor_Tantalum_SMD:CP_EIA-7343-31_Kemet-D_Pad2.25x2.55mm_HandSolder -> Capacitor_SMD:C_0805_2012Metric
- C17: value 587-5514-1-ND -> 680pF; footprint Capacitor_SMD:C_0402_1005Metric -> Capacitor_SMD:C_0805_2012Metric
- C18: value 587-5514-1-ND -> 10uF; footprint Capacitor_SMD:C_0402_1005Metric -> Capacitor_SMD:C_1206_3216Metric
- C19, C20: value 311-3342-1-ND -> 10uF; footprint Capacitor_SMD:C_0402_1005Metric -> Capacitor_SMD:C_1206_3216Metric
- C2, C4: value 587-5514-1-ND -> 22uF; footprint Capacitor_SMD:C_0402_1005Metric -> Capacitor_SMD:C_2220_5650Metric
- C21, C9: value 311-3342-1-ND -> 1uF
- C22: value 311-3342-1-ND -> 10uF; footprint Capacitor_SMD:C_0402_1005Metric -> Capacitor_SMD:C_0805_2012Metric
- C23: value 311-3342-1-ND -> 6.8pF
- C24: value 1uF -> 0.1uF
- C25: value 1uF -> 6.8pF
- C27, C35, C44, C49, C50: value 1uF -> 587-5514-1-ND
- C28: value 220uF -> 587-5514-1-ND; footprint Capacitor_SMD:CP_Elec_6.3x7.7 -> Capacitor_SMD:C_0402_1005Metric; moved to F.Cu
- C29: value 311-3342-1-ND -> 587-5514-1-ND
- C3: value 587-5514-1-ND -> ~
- C30, C31: value 6.8pF -> 587-5514-1-ND
- C32: value 470pF -> 311-3342-1-ND
- C34, C36: value 47uF -> 311-3342-1-ND; footprint Capacitor_SMD:C_1210_3225Metric -> Capacitor_SMD:C_0402_1005Metric
- C37: value 47uF -> 587-5514-1-ND; footprint Capacitor_SMD:C_1210_3225Metric -> Capacitor_SMD:C_0402_1005Metric
- C38: value 1uF -> 587-5514-1-ND; footprint Capacitor_SMD:C_0805_2012Metric -> Capacitor_SMD:C_0402_1005Metric
- C39: value 3.3nF -> 1uF
- C40: value 180pF -> 1uF; footprint Capacitor_SMD:C_0805_2012Metric -> Capacitor_SMD:C_0402_1005Metric
- C41: value 1.5nF -> 587-5514-1-ND; footprint Capacitor_SMD:C_0805_2012Metric -> Capacitor_SMD:C_0402_1005Metric
- C42: value 0.1uF -> 330uF; footprint Capacitor_SMD:C_0402_1005Metric -> Capacitor_Tantalum_SMD:CP_EIA-7343-31_Kemet-D_Pad2.25x2.55mm_HandSolder
- C43, C51: value 10uF -> 587-5514-1-ND; footprint Capacitor_SMD:C_0805_2012Metric -> Capacitor_SMD:C_0402_1005Metric
- C45: value 470pF -> 587-5514-1-ND; footprint Capacitor_SMD:C_0805_2012Metric -> Capacitor_SMD:C_0402_1005Metric
- C46: value 220uF -> 587-5514-1-ND; footprint TPS40305_supply:CAP_2R5TPE220MAFB -> Capacitor_SMD:C_0402_1005Metric
- C47: value 100uF -> 587-5514-1-ND; footprint Capacitor_SMD:C_1206_3216Metric -> Capacitor_SMD:C_0402_1005Metric
- C5: value 587-5514-1-ND -> 1uF; footprint Capacitor_SMD:C_0402_1005Metric -> Capacitor_SMD:C_0805_2012Metric
- C52: value 0.1uF -> 587-5514-1-ND
- C6: value 587-5514-1-ND -> 3.3nF
- C7: value 311-3342-1-ND -> 270pF; footprint Capacitor_SMD:C_0402_1005Metric -> Capacitor_SMD:C_0805_2012Metric
- C8: value 587-5514-1-ND -> 5.6nF; footprint Capacitor_SMD:C_0402_1005Metric -> Capacitor_SMD:C_0805_2012Metric
- J4: footprint bitaxe:470531000 -> Connector_PinHeader_2.54mm:PinHeader_1x04_P2.54mm_Vertical
- J5: moved to F.Cu
- J6: value Conn_01x08 -> Conn_01x04; footprint Connector_PinHeader_2.54mm:PinHeader_1x08_P2.54mm_Vertical -> bitaxe:470531000
- J7: value Conn_01x02 -> Conn_01x04; footprint Connector_PinHeader_2.54mm:PinHeader_1x02_P2.54mm_Vertical -> bitaxe:470531000
- L1: value 150nH -> 470nH; footprint TPS40305_supply:FP1005R1-R15-R -> bitaxe:744373580047
- Q1: value CSD17311Q5 -> NTMFS5C673NLT1G; footprint TPS40305_supply:CSD17311Q5 -> bitaxe:NTMFS5C673NLT1G
- Q2: value CSD17311Q5 -> CSD17577Q5A; footprint TPS40305_supply:CSD17311Q5 -> bitaxe:CSD17577Q5A
- R1: value 1k -> 2m; footprint Resistor_SMD:R_0402_1005Metric -> Resistor_SMD:R_1206_3216Metric
- R10: value 3.83k -> DNP
- R11: value 100k -> 10k
- R12: value 4.12k -> 1.54k
- R13: value 1.33k -> 10k
- R14: value 4.99k -> 1k
- R15: value 3.32k -> 1k
- R16: value 80k -> 0
- R17: value DNP -> 0
- R18: value 1k -> 0
- R19: value 1k -> 1; footprint Resistor_SMD:R_0402_1005Metric -> Resistor_SMD:R_2512_6332Metric
- R20, R36: value 10k -> 1; footprint Resistor_SMD:R_0402_1005Metric -> Resistor_SMD:R_2512_6332Metric
- R21, R22: value 60.4 -> 0
- R24: value 10k -> 100
- R25: value 19.1k -> 100
- R28, R29: value 261 -> 10k
- R4: value 10k -> 1.33k
- R5: value 0 -> 10k
- R6: value 10k -> 100k
- R7: value 100 -> 6.49k
- R8: value 100 -> 80k
- R9: value 10k -> 487
- U1: value 25MHz -> INA219AIDCNR; footprint bitaxe:O 25,0-JO32-B-1V3-1-T1-LF -> lcsc:SOT-23-8_L3.0-W1.7-P0.65-LS2.8-BR
- U10: value DS4432U+ -> EMC2101
- U11: value RT9080-33GJ5 -> MCP1824T-1802E; footprint bitaxe:RT9080-33GJ5 -> Package_TO_SOT_SMD:SOT-23-5
- U12: value ESP32-S3-WROOM-1 -> MCP1824T-0802E; footprint Espressif:ESP32-S3-WROOM-1 -> Package_TO_SOT_SMD:SOT-23-5; moved to F.Cu
- U13: value CLX6E-FKC -> MCP1824T-1802E; footprint bitaxe:CLX6E-FKC-CH1M1D1BB7C3D3 -> Package_TO_SOT_SMD:SOT-23-5; moved to F.Cu
- U2: value TXB0104RGYR -> TPS40305; footprint bitaxe:TXB0104 -> TPS40305_supply:TPS40305
- U3: value SN74AXC1T45DBVR -> uA7805; footprint bitaxe:SN74AXC1T45 -> Package_TO_SOT_SMD:TO-263-2
- U4: value CLX6E-FKC -> RT9080-33GJ5; footprint bitaxe:CLX6E-FKC-CH1M1D1BB7C3D3 -> bitaxe:RT9080-33GJ5; moved to F.Cu
- U5: value MCP1824 -> DS4432U+; footprint Package_TO_SOT_SMD:SOT-23-5 -> Package_SO:TSSOP-8_3x3mm_P0.65mm
- U6: value MCP1824 -> ESP32-S3-WROOM-1; footprint Package_TO_SOT_SMD:SOT-23-5 -> Espressif:ESP32-S3-WROOM-1
- U7: value EMC2101 -> MCP1824T-1802E; footprint Package_SO:TSSOP-8_3x3mm_P0.65mm -> Package_TO_SOT_SMD:SOT-23-5
- U8: value INA260 -> MCP1824T-0802E; footprint Package_SO:TSSOP-16_4.4x5mm_P0.65mm -> Package_TO_SOT_SMD:SOT-23-5
- U9: value TPS40305 -> EMC2101; footprint TPS40305_supply:TPS40305 -> Package_SO:TSSOP-8_3x3mm_P0.65mm
- moved U3 186.6 mm to (-50.7, 146.0)
- moved J4 162.2 mm to (-69.1, 110.1)
- moved C51 151.4 mm to (-19.6, 70.8)
- moved U9 151.3 mm to (-52.6, 56.2), turned to 0 degrees
- moved U7 149.0 mm to (-66.5, 120.5)
- moved J5 147.6 mm to (-18.0, 36.8), turned to 0 degrees
- moved R25 147.1 mm to (-56.3, 126.8)
- moved C45 147.0 mm to (-54.2, 51.5)
- moved U13 147.0 mm to (-34.5, 35.0), turned to 0 degrees
- moved U4 146.7 mm to (-45.1, 35.8), turned to 0 degrees
- moved U2 146.6 mm to (-22.2, 92.4)
- moved C10 146.6 mm to (-35.4, 98.5)
- moved C11 146.6 mm to (-44.3, 98.5)
- moved C15 146.6 mm to (-47.7, 89.9)
- moved C17 146.6 mm to (-48.9, 91.7)
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Connections:
- C1 pad 1: GND -> /Power/VIN_M
- C1 pad 2: /BM1397/1V8 -> GND
- C10 pad 1: /VDD -> /Power/VIN_M
- C11 pad 1: /VDD -> /5V
- C12 pad 1: /VDD -> Net-(U2-BOOT)
- C12 pad 2: Net-(C12-Pad2) -> /Power/SW
- C13 pad 1: /VDD -> Net-(U2-BP)
- C14 pad 1: /BM1397/1V8 -> /5V
- C15 pad 1: Net-(C12-Pad2) -> /3V3
- C15 pad 2: Net-(C15-Pad2) -> GND
- C16 pad 1: /BM1397/0V8 -> /3V3
- C17 pad 1: Net-(C15-Pad2) -> Net-(C17-Pad1)
- C17 pad 2: Net-(C17-Pad2) -> /Power/OUT0
- C18 pad 1: Net-(C17-Pad2) -> /VDD
- C19 pad 1: /BM1397/1V8 -> /VDD
- C2 pad 1: GND -> /Power/VIN_M
- C2 pad 2: Net-(C2-Pad2) -> GND
- C20 pad 1: /3V3 -> /VDD
- C21 pad 1: /BM1397/1V8 -> /ESP32/EN
- C22 pad 1: /5V -> /ESP32/3V3
- C23 pad 1: /5V -> /ESP32/XIN32
- C24 pad 1: /BM1397/1V8 -> /ESP32/3V3
- C25 pad 1: /BM1397/0V8 -> /ESP32/XOUT32
- C26 pad 1: /3V3 -> GND
- C26 pad 2: GND -> /BM1397-1/1V8
- C27 pad 1: /5V -> GND
- C27 pad 2: GND -> Net-(IC1-VDD1_0)
- C28 pad 1: /5V -> Net-(IC1-VDD1_0)
- C28 pad 2: GND -> Net-(IC1-VDD2_0)
- C29 pad 1: /5V -> /BM1397-1/0V8
- C3 pad 1: Net-(C2-Pad2) -> Net-(U1-IN+)
- C3 pad 2: Net-(C3-Pad2) -> Net-(U1-IN-)
- C30 pad 1: /ESP32/XIN32 -> /BM1397-1/1V8
- C31 pad 1: /ESP32/XOUT32 -> Net-(IC1-VDD2_0)
- C31 pad 2: GND -> Net-(IC1-VDD3_0)
- C32 pad 1: Net-(C32-Pad1) -> /5V
- C32 pad 2: Net-(C32-Pad2) -> GND
- C33 pad 1: /3V3 -> /5V
- C34 pad 1: /5V -> /VDD
- C35 pad 1: /3V3 -> Net-(IC1-VDD3_0)
- C35 pad 2: GND -> /VDD
- C36 pad 1: /5V -> /VDD
- C37 pad 1: /5V -> /VDD
- C38 pad 1: /5V -> /VDD
- C39 pad 1: Net-(C39-Pad1) -> /BM1397-1/1V8
- C4 pad 1: /BM1397/0V8 -> /Power/VIN_M
- C40 pad 1: Net-(C40-Pad1) -> /BM1397-1/0V8
- C40 pad 2: /Power/OUT0 -> GND
- C41 pad 1: Net-(C40-Pad1) -> /VDD
- C41 pad 2: Net-(C41-Pad2) -> Net-(IC1-VDD3_1)
- C42 pad 1: Net-(C42-Pad1) -> /VDD
- C42 pad 2: /Power/SW -> GND
- C43 pad 1: Net-(C43-Pad1) -> Net-(IC1-VDD3_1)
- C43 pad 2: GND -> Net-(IC1-VDD2_1)
- C44 pad 1: /3V3 -> /BM1397-1/1V8
- C45 pad 1: Net-(C45-Pad1) -> /BM1397-1/0V8
- C45 pad 2: /Power/OUT0 -> GND
- C46 pad 1: /VDD -> Net-(IC1-VDD2_1)
- C46 pad 2: GND -> Net-(IC1-VDD1_1)
- C47 pad 1: /VDD -> Net-(IC1-VDD1_1)
- C49 pad 1: /3V3 -> Net-(IC2-VDD1_0)
- C49 pad 2: GND -> Net-(IC2-VDD2_0)
- C5 pad 1: /BM1397/1V8 -> /Power/VIN_M
- C50 pad 1: /ESP32/EN -> /BM1397-1/0V8
- C51 pad 1: /3V3 -> /BM1397-1/1V8
- C52 pad 1: /3V3 -> Net-(IC2-VDD2_0)
- C52 pad 2: GND -> Net-(IC2-VDD3_0)
- C6 pad 1: Net-(C3-Pad2) -> Net-(U2-SS)
- C6 pad 2: Net-(C6-Pad2) -> GND
- C7 pad 1: /VDD -> Net-(U2-COMP)
- C7 pad 2: GND -> /Power/OUT0
- C8 pad 1: Net-(C6-Pad2) -> Net-(U2-COMP)
- C8 pad 2: /VDD -> Net-(C8-Pad2)
- C9 pad 1: /VDD -> /3V3
- IC1 pad 1: Net-(C6-Pad2) -> Net-(IC1-VDD3_0)
- IC1 pad 10: Net-(IC1-Pad10) -> /RO
- IC1 pad 11: Net-(IC1-Pad11) -> /CI
- IC1 pad 12: /BM1397/BM_CLKI -> Net-(IC1-CLKI)
- IC1 pad 14: /BM1397/0V8 -> /BM1397-1/0V8
- IC1 pad 15: /BM1397/0V8 -> /BM1397-1/0V8
- IC1 pad 16: /BM1397/1V8 -> /BM1397-1/1V8
- IC1 pad 17: /BM1397/1V8 -> /BM1397-1/1V8
- IC1 pad 18: /BM1397/0V8 -> /BM1397-1/0V8
- IC1 pad 2: Net-(C3-Pad2) -> Net-(IC1-VDD2_0)
- IC1 pad 20: Net-(IC1-Pad20) -> unconnected-(IC1-PIN_MODE-Pad20)
- IC1 pad 21: /TEMP_N -> unconnected-(IC1-TEMP_N-Pad21)
- IC1 pad 22: /TEMP_P -> unconnected-(IC1-TEMP_P-Pad22)
- IC1 pad 25: Net-(IC1-Pad25) -> Net-(IC1-CLKO)
- IC1 pad 26: Net-(IC1-Pad26) -> Net-(IC1-CO)
- IC1 pad 27: Net-(IC1-Pad27) -> Net-(IC1-RI)
- IC1 pad 28: Net-(IC1-Pad28) -> Net-(IC1-NRSTO)
- IC1 pad 29: Net-(IC1-Pad29) -> Net-(IC1-BO)
- IC1 pad 3: Net-(C2-Pad2) -> Net-(IC1-VDD1_0)
- IC1 pad 30: Net-(C17-Pad2) -> Net-(IC1-VDD1_1)
- IC1 pad 31: Net-(C15-Pad2) -> Net-(IC1-VDD2_1)
- IC1 pad 32: Net-(C12-Pad2) -> Net-(IC1-VDD3_1)
- IC1 pad 4: Net-(IC1-Pad4) -> Net-(IC1-ADDR0)
- IC1 pad 5: Net-(IC1-Pad5) -> Net-(IC1-ADDR1)
- IC1 pad 6: Net-(IC1-Pad6) -> Net-(IC1-ADDR2)
- IC1 pad 8: /BM1397/BM_BI -> unconnected-(IC1-BI-Pad8)
- IC1 pad 9: /BM1397/RST_N -> /NRSTI
- J4 pad 2: /5V -> /ESP32/3V3
- J4 pad 3: /Fan/FAN_TACH -> /SCL
- J4 pad 4: /Fan/FAN_PWM -> /SDA
- J5 pad 2: /3V3 -> /ESP32/3V3
- J6 pad 1: /BI -> GND
- J6 pad 2: /RST -> /5V
- J6 pad 3: /RX -> /Fan/FAN_TACH1
- J6 pad 4: /TX -> /Fan/FAN_PWM1
- J7 pad 1: /Power/VIN -> GND
- Q1 pad 4: Net-(Q1-Pad4) -> Net-(Q1-G)
- Q1 pad 5: /5V -> /Power/VIN_M
- Q2 pad 4: Net-(Q2-Pad4) -> Net-(Q2-G)
- R1 pad 1: GND -> /Power/VIN
- R1 pad 2: /BM1397/RST_N -> /Power/VIN_M
- R10 pad 1: Net-(C41-Pad2) -> Net-(U5-FS1)
- R10 pad 2: /Power/OUT0 -> GND
- R11 pad 1: /Power/PGOOD -> /VDD
- R11 pad 2: Net-(C43-Pad1) -> /Power/OUT0
- R12 pad 1: Net-(Q2-Pad4) -> /Power/OUT0
- R13 pad 1: /VDD -> /ESP32/3V3
- R13 pad 2: Net-(C45-Pad1) -> /ESP32/EN
- R14 pad 1: /VDD -> /SCL
- R14 pad 2: /Power/OUT0 -> /ESP32/3V3
- R15 pad 1: /Power/OUT0 -> /SDA
- R15 pad 2: GND -> /ESP32/3V3
- R16 pad 1: Net-(R16-Pad1) -> GND
- R16 pad 2: GND -> Net-(IC1-ADDR0)
- R17 pad 1: Net-(R17-Pad1) -> GND
- R17 pad 2: GND -> Net-(IC1-ADDR1)
- R18 pad 1: /SCL -> GND
- R18 pad 2: /3V3 -> Net-(IC1-ADDR2)
- R19 pad 1: /SDA -> /VDD
- R19 pad 2: /3V3 -> GND
- R2 pad 1: Net-(R2-Pad1) -> /Power/VIN
- R2 pad 2: /BM1397/BM_CLKI -> Net-(U1-IN+)
- R20 pad 1: /3V3 -> /VDD
- R20 pad 2: /ESP32/EN -> GND
- R21 pad 1: /ESP32/LEDX_B -> GND
- R21 pad 2: Net-(R21-Pad2) -> Net-(IC2-ADDR0)
- R22 pad 1: /ESP32/LEDZ_B -> GND
- R22 pad 2: Net-(R22-Pad2) -> Net-(IC2-ADDR1)
- R23 pad 1: /BM1397/BM_CLKI -> GND
- R23 pad 2: Net-(R23-Pad2) -> Net-(IC2-ADDR2)
- R24 pad 1: /ESP32/FAN_ALERT -> Net-(U9-DN)
- R24 pad 2: /Fan/FAN_TACH -> /TEMP1_N
- R25 pad 1: GND -> Net-(U10-DN)
- R25 pad 2: /ESP32/FAN_ALERT -> /TEMP2_N
- R26 pad 1: /ESP32/LEDX_G -> /TEMP1_P
- R26 pad 2: Net-(R26-Pad2) -> Net-(U9-DP)
- R27 pad 1: /ESP32/LEDZ_G -> /TEMP2_P
- R27 pad 2: Net-(R27-Pad2) -> Net-(U10-DP)
- R28 pad 1: /ESP32/LEDX_R -> /Fan/FAN_PWM1
- R28 pad 2: Net-(R28-Pad2) -> /3V3
- R29 pad 1: /ESP32/LEDZ_R -> /Fan/FAN_PWM2
- R29 pad 2: Net-(R29-Pad2) -> /3V3
- R3 pad 1: /BM1397/RO -> /Power/VIN_M
- R3 pad 2: Net-(IC1-Pad10) -> Net-(U1-IN-)
- R36 pad 1: /Fan/FAN_TACH -> GND
- R36 pad 2: /3V3 -> GND
- R4 pad 1: /3V3 -> Net-(C8-Pad2)
- R4 pad 2: /Power/PGOOD -> /Power/OUT0
- R5 pad 1: /BM1397/CI -> /3V3
- R5 pad 2: Net-(IC1-Pad11) -> /Power/PGOOD
- R6 pad 1: Net-(IC1-Pad27) -> /Power/PGOOD
- R6 pad 2: /BM1397/1V8 -> Net-(U2-BP)
- R7 pad 1: Net-(C32-Pad2) -> Net-(Q2-G)
- R7 pad 2: /TEMP_N -> GND
- R8 pad 1: /TEMP_P -> Net-(U5-FS0)
- R8 pad 2: Net-(C32-Pad1) -> GND
- R9 pad 1: /Fan/FAN_PWM -> /VDD
- R9 pad 2: /3V3 -> Net-(C17-Pad1)
- TP1 pad 1: Net-(R2-Pad1) -> /ESP32/3V3
- TP10 pad 1: Net-(IC1-Pad20) -> /Fan/FAN_TACH1
- TP11 pad 1: /TEMP_P -> /Fan/FAN_TACH2
- TP12 pad 1: /TEMP_N -> /Fan/FAN_PWM1
- TP13 pad 1: /BM1397/1V8 -> /Fan/FAN_PWM2
- TP14 pad 1: /BM1397/0V8 -> /BM1398-2/1V8
- TP15 pad 1: /Fan/FAN_PWM -> Net-(IC3-PIN_MODE)
- TP16 pad 1: /Fan/FAN_TACH -> /BM1398-2/0V8
- TP17 pad 1: /ESP32/EN -> /TEMP1_P
- TP18 pad 1: /ESP32/P_TX -> /TEMP1_N
- TP19 pad 1: /3V3 -> Net-(IC4-PIN_MODE)
- TP2 pad 1: /BM1397/CI -> GND
- TP21 pad 1: /BM1397/CLKI -> /TEMP2_N
- TP22 pad 1: /ESP32/P_RX -> /BM1397-3/1V8
- TP23 pad 1: /ESP32/IO0 -> /BM1397-3/0V8
- TP24 pad 1: /BM1397/BM_BI -> Net-(IC6-BO)
- TP25 pad 1: /ESP32/LEDX_R -> Net-(IC6-NRSTO)
- TP26 pad 1: /ESP32/LEDX_G -> Net-(IC6-RI)
- TP27 pad 1: /ESP32/LEDX_B -> Net-(IC6-CO)
- TP28 pad 1: /ESP32/LEDZ_R -> Net-(IC6-CLKO)
- TP3 pad 1: /BM1397/RO -> /ESP32/EN
- TP4 pad 1: /BM1397/RST_N -> /ESP32/P_TX
- TP5 pad 1: GND -> /ESP32/P_RX
- TP6 pad 1: Net-(IC1-Pad29) -> /ESP32/IO0
- TP7 pad 1: Net-(IC1-Pad28) -> Net-(IC1-CLKI)
- TP8 pad 1: Net-(IC1-Pad26) -> /BM1397-1/1V8
- TP9 pad 1: Net-(IC1-Pad25) -> /BM1397-1/0V8
- U1 pad 1: /BM1397/1V8 -> Net-(U1-IN+)
- U1 pad 2: GND -> Net-(U1-IN-)
- U1 pad 3: Net-(R2-Pad1) -> GND
- U1 pad 4: /BM1397/1V8 -> /3V3
- U10 pad 1: /SDA -> /3V3
- U10 pad 2: /SCL -> Net-(U10-DP)
- U10 pad 3: Net-(R17-Pad1) -> Net-(U10-DN)
- U10 pad 4: GND -> /Fan/FAN_PWM2
- U10 pad 5: Net-(R16-Pad1) -> GND
- U10 pad 6: /Power/OUT0 -> /Fan/FAN_TACH2
- U10 pad 7: /Power/OUT1 -> /SDA
- U10 pad 8: /3V3 -> /SCL
- U11 pad 4: (no net) -> unconnected-(U11-PG-Pad4)
- U11 pad 5: /3V3 -> /BM1398-2/1V8
- U12 pad 1: GND -> /5V
- U12 pad 2: /3V3 -> GND
- U12 pad 3: /ESP32/EN -> /5V
- U12 pad 5: /ESP32/LEDZ_R -> /BM1398-2/0V8
- U13 pad 1: GND -> /5V
- U13 pad 3: GND -> /5V
- U13 pad 4: Net-(R29-Pad2) -> unconnected-(U13-PG-Pad4)
- U13 pad 5: Net-(R27-Pad2) -> /BM1397-3/1V8
- U2 pad 1: /BM1397/1V8 -> /Power/VIN_M
- U2 pad 10: /BI -> Net-(U2-BP)
- U2 pad 11: /RST -> GND
- U2 pad 2: /BM1397/RO -> Net-(U2-SS)
- U2 pad 3: /BM1397/CI -> /Power/PGOOD
- U2 pad 4: /BM1397/RST_N -> Net-(U2-COMP)
- U2 pad 5: /BM1397/BM_BI -> /Power/OUT0
- U2 pad 6: (no net) -> Net-(U2-BOOT)
- U2 pad 7: GND -> Net-(Q1-G)
- U2 pad 8: /BM1397/1V8 -> /Power/SW
- U2 pad 9: (no net) -> Net-(Q2-G)
- U3 pad 1: /BM1397/1V8 -> /Power/VIN_M
- U3 pad 3: Net-(R23-Pad2) -> /5V
- U4 pad 1: GND -> /5V
- U4 pad 3: GND -> /5V
- U4 pad 4: Net-(R28-Pad2) -> (no net)
- U4 pad 5: Net-(R26-Pad2) -> /3V3
- U5 pad 1: /5V -> /SDA
- U5 pad 2: GND -> /SCL
- U5 pad 3: /5V -> Net-(U5-FS1)
- U5 pad 4: unconnected-(U5-Pad4) -> GND
- U5 pad 5: /BM1397/1V8 -> Net-(U5-FS0)
- U6 pad 1: /5V -> GND
- U6 pad 2: GND -> /ESP32/3V3
- U6 pad 3: /5V -> /ESP32/EN
- U6 pad 5: /BM1397/0V8 -> unconnected-(U6-GPIO5/TOUCH5/ADC1_CH4-Pad5)
- U7 pad 1: /3V3 -> /5V
- U7 pad 2: Net-(C32-Pad1) -> GND
- U7 pad 3: Net-(C32-Pad2) -> /5V
- U7 pad 4: /Fan/FAN_PWM -> unconnected-(U7-PG-Pad4)
- U7 pad 5: GND -> /BM1397-1/1V8
- U8 pad 1: /Power/VIN -> /5V
- U8 pad 2: /Power/VIN -> GND
- U8 pad 3: /Power/VIN -> /5V
- U8 pad 4: GND -> unconnected-(U8-PG-Pad4)
- U8 pad 5: GND -> /BM1397-1/0V8
- U9 pad 1: /5V -> /3V3
- U9 pad 2: Net-(C39-Pad1) -> Net-(U9-DP)
- U9 pad 3: /Power/PGOOD -> Net-(U9-DN)
- U9 pad 4: Net-(C40-Pad1) -> /Fan/FAN_PWM1
- U9 pad 5: /Power/OUT0 -> GND
- U9 pad 6: Net-(C42-Pad1) -> /Fan/FAN_TACH1
- U9 pad 7: Net-(Q1-Pad4) -> /SDA
- U9 pad 8: /Power/SW -> /SCL
Routing:
- net /5V: track 180.2 -> 0.00 mm, vias 6 -> 0
- net /SDA: track 175.0 -> 0.00 mm, vias 6 -> 0
- net /SCL: track 161.0 -> 0.00 mm, vias 5 -> 0
- net GND: track 133.4 -> 0.00 mm, vias 73 -> 0
- net /BM1397/1V8: track 128.5 -> 0.00 mm, vias 6 -> 0
- net /ESP32/FAN_ALERT: track 112.3 -> 0.00 mm, vias 3 -> 0
- net /RST: track 89.2 -> 0.00 mm, vias 2 -> 0
- net /VDD: track 83.9 -> 0.00 mm, vias 19 -> 0
- net /3V3: track 82.9 -> 0.00 mm, vias 16 -> 0
- net /BI: track 77.5 -> 0.00 mm, vias 2 -> 0
- net /RX: track 73.8 -> 0.00 mm, vias 1 -> 0
- net /TX: track 72.7 -> 0.00 mm, vias 1 -> 0
- net /BM1397/RST_N: track 70.9 -> 0.00 mm, vias 2 -> 0
- net /BM1397/CI: track 64.7 -> 0.00 mm, vias 2 -> 0
- net /BM1397/RO: track 60.6 -> 0.00 mm, vias 2 -> 0
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- removed copper zone on F.Cu, net /5V
- removed copper zone on F.Cu, net /Power/SW
- removed copper zone on F.Cu, net /Power/VIN
- removed copper zone on B.Cu, net /VDD
- removed copper zone on F.Cu, net /VDD
- removed copper zone on B.Cu, net GND
- removed copper zone on F.Cu, net GND
Other:
- board size 56.5 x 99.8 mm -> 136.3 x 79.7 mm
- board text removed: "3V3"
- board text removed: "5V"
- board text removed: "BI"
- board text removed: "BM1397 V2.2"
- board text removed: "PWM"
- board text removed: "RX"
- board text removed: "SCL"
- board text removed: "SDA"
- board text removed: "TAC"
- board text removed: "TX"

Commit message: some more placements, added level shifters..
Parts:
- removed R43, R44: 1, Resistor_SMD:R_2512_6332Metric
- removed TP15, TP17, TP18, TP19: TestPoint, TestPoint:TestPoint_Pad_D1.5mm
- added C149: 470pF, Capacitor_SMD:C_0402_1005Metric, F.Cu at (-55.7, 10.6)
- added C150: 311-3342-1-ND, Capacitor_SMD:C_0402_1005Metric, F.Cu at (-55.7, 12.6)
- added C151: 220uF, Capacitor_SMD:CP_Elec_6.3x7.7, B.Cu at (165.7, 123.0)
- added C152: 311-3342-1-ND, Capacitor_SMD:C_0402_1005Metric, F.Cu at (-55.7, 14.6)
- added C153: 311-3342-1-ND, Capacitor_SMD:C_0402_1005Metric, F.Cu at (-9.28, 121.6)
- added C154: 311-3342-1-ND, Capacitor_SMD:C_0402_1005Metric, F.Cu at (-9.28, 123.6)
- added C155: 311-3342-1-ND, Capacitor_SMD:C_0402_1005Metric, F.Cu at (-9.28, 125.6)
- added C156: 311-3342-1-ND, Capacitor_SMD:C_0402_1005Metric, F.Cu at (-9.28, 127.5)
- added C157: 311-3342-1-ND, Capacitor_SMD:C_0402_1005Metric, F.Cu at (-9.28, 129.5)
- added C158: 311-3342-1-ND, Capacitor_SMD:C_0402_1005Metric, F.Cu at (-9.28, 131.5)
- added G***: LOGO, LOGO, F.Cu at (217.9, 51.3)
- added J3: Conn_01x04, bitaxe:470531000, B.Cu at (181.4, 122.4)
- added J8: Conn_01x05, Connector_PinHeader_2.54mm:PinHeader_1x05_P2.54mm_Vertical, F.Cu at (-7.66, 10.1)
- added R48: 100, Resistor_SMD:R_0402_1005Metric, F.Cu at (-62.2, 10.7)
- added R49: 100, Resistor_SMD:R_0402_1005Metric, F.Cu at (-62.2, 12.6)
- added R50: 10k, Resistor_SMD:R_0402_1005Metric, F.Cu at (-62.2, 14.6)
- added R51: 5.6k, Resistor_SMD:R_0402_1005Metric, F.Cu at (-62.2, 16.6)
- added TP29: TestPoint, TestPoint:TestPoint_Pad_D1.5mm, F.Cu at (-58.9, 11.4)
- added TP30: TestPoint, TestPoint:TestPoint_Pad_D1.5mm, F.Cu at (-58.9, 15.0)
- added TP31: TestPoint, TestPoint:TestPoint_Pad_D1.5mm, F.Cu at (-72.3, 21.6)
- added TP32: TestPoint, TestPoint:TestPoint_Pad_D1.5mm, F.Cu at (-72.3, 25.1)
- added TP33: TestPoint, TestPoint:TestPoint_Pad_D1.5mm, F.Cu at (-66.7, 21.6)
- added TP34: TestPoint, TestPoint:TestPoint_Pad_D1.5mm, F.Cu at (-66.7, 25.1)
- added U15: EMC2101, Package_SO:TSSOP-8_3x3mm_P0.65mm, F.Cu at (-58.8, 4.32)
- added U16: SN74LVC1T45DBVR, lcsc:SOT-23-6_L2.9-W1.6-P0.95-LS2.8-BR, F.Cu at (-13.1, 122.8)
- added U17: SN74LVC1T45DBVR, lcsc:SOT-23-6_L2.9-W1.6-P0.95-LS2.8-BR, F.Cu at (-13.1, 127.4)
- added U18: SN74LVC1T45DBVR, lcsc:SOT-23-6_L2.9-W1.6-P0.95-LS2.8-BR, F.Cu at (-13.1, 132.0)
- C69, C70, SW1, SW2, U6, USB1: moved to B.Cu
- moved USB1 253.6 mm to (186.2, 59.8), turned to -90 degrees
- moved SW2 253.5 mm to (185.4, 72.4), turned to 180 degrees
- moved SW1 253.5 mm to (185.4, 68.2), turned to 180 degrees
- moved C143 235.7 mm to (183.4, 100.0), turned to -90 degrees
- moved R35 226.9 mm to (143.3, 88.5)
- moved C126 214.4 mm to (162.7, 100.0), turned to -90 degrees
- moved C105 211.4 mm to (139.7, 99.2), turned to 90 degrees
- moved R36 197.9 mm to (143.5, 84.1)
- moved C88 190.9 mm to (119.5, 99.1), turned to 90 degrees
- moved C59 185.8 mm to (95.5, 100.0), turned to -90 degrees
- moved C70 183.0 mm to (121.7, 123.2), turned to 180 degrees
- moved C69 141.0 mm to (76.9, 123.0), turned to 180 degrees
- moved R19 129.2 mm to (100.1, 84.3)
- moved R20 117.7 mm to (100.1, 89.0), turned to 0 degrees
- moved C42 96.9 mm to (77.5, 99.8), turned to -90 degrees
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Connections:
- net /BM1397-1/1V8 renamed /1V8
- C100 pad 2: GND -> /BM1397-1/GND1
- C101 pad 1: GND -> /BM1397-1/GND1
- C101 pad 2: GND -> /BM1397-3/VDD3
- C102 pad 1: GND -> /BM1397-1/GND1
- C102 pad 2: GND -> /BM1397-3/VDD3
- C103 pad 1: GND -> /BM1397-1/GND1
- C103 pad 2: GND -> /BM1397-3/VDD3
- C104 pad 1: GND -> /BM1397-1/GND1
- C105 pad 1: GND -> /BM1397-1/GND1
- C105 pad 2: GND -> /BM1397-3/VDD3
- C107 pad 2: GND -> /BM1397-3/VDD3
- C108 pad 2: GND -> /BM1397-3/VDD3
- C110 pad 2: GND -> /BM1397-3/VDD3
- C116 pad 1: GND -> /BM1397-3/VDD3
- C119 pad 2: GND -> /BM1397-3/VDD3
- C120 pad 1: GND -> /BM1397-3/VDD3
- C121 pad 1: GND -> /BM1397-3/VDD3
- C122 pad 1: GND -> /BM1397-3/VDD3
- C125 pad 1: GND -> /BM1397-3/VDD3
- C126 pad 1: GND -> /BM1397-3/VDD3
- C137 pad 1: GND -> /BM1397-3/VDD3
- C138 pad 2: GND -> /BM1397-3/VDD3
- C139 pad 1: GND -> /BM1397-3/VDD3
- C140 pad 1: GND -> /BM1397-3/VDD3
- C141 pad 1: GND -> /BM1397-3/VDD3
- C142 pad 1: GND -> /BM1397-3/VDD3
- C143 pad 1: GND -> /BM1397-3/VDD3
- C22 pad 1: /ESP32/3V3 -> /3V3
- C24 pad 1: /ESP32/3V3 -> /3V3
- C26 pad 1: GND -> /BM1397-1/GND1
- C27 pad 1: GND -> /BM1397-1/GND1
- C29 pad 2: GND -> /BM1397-1/GND1
- C30 pad 2: GND -> /BM1397-1/GND1
- C32 pad 2: GND -> /BM1397-1/GND1
- C33 pad 2: GND -> /BM1397-1/GND1
- C34 pad 2: GND -> /BM1397-1/GND1
- C36 pad 2: GND -> /BM1397-1/GND1
- C37 pad 2: GND -> /BM1397-1/GND1
- C38 pad 2: GND -> /BM1397-1/GND1
- C39 pad 2: GND -> /BM1397-1/GND1
- C40 pad 2: GND -> /BM1397-1/GND1
- C42 pad 2: GND -> /BM1397-1/GND1
- C44 pad 2: GND -> /BM1397-1/GND1
- C45 pad 2: GND -> /BM1397-1/GND1
- C47 pad 2: GND -> /BM1397-1/GND1
- C48 pad 1: GND -> /BM1397-1/GND1
- C50 pad 2: GND -> /BM1397-1/GND1
- C51 pad 2: GND -> /BM1397-1/GND1
- C53 pad 2: GND -> /BM1397-1/GND1
- C55 pad 2: GND -> /BM1397-1/GND1
- C56 pad 2: GND -> /BM1397-1/GND1
- C57 pad 2: GND -> /BM1397-1/GND1
- C59 pad 2: GND -> /BM1397-1/GND1
- C61 pad 2: GND -> /BM1397-1/GND1
- C62 pad 2: GND -> /BM1397-1/GND1
- C64 pad 2: GND -> /BM1397-1/GND1
- C73 pad 1: GND -> /BM1397-3/VDD3
- C75 pad 2: GND -> /BM1397-3/VDD3
- C76 pad 2: GND -> /BM1397-3/VDD3
- C78 pad 1: GND -> /BM1397-1/GND1
- C78 pad 2: GND -> /BM1397-3/VDD3
- C79 pad 2: GND -> /BM1397-3/VDD3
- C80 pad 2: GND -> /BM1397-3/VDD3
- C81 pad 2: GND -> /BM1397-1/GND1
- C82 pad 1: GND -> /BM1397-1/GND1
- C82 pad 2: GND -> /BM1397-3/VDD3
- C83 pad 1: GND -> /BM1397-1/GND1
- C83 pad 2: GND -> /BM1397-3/VDD3
- C84 pad 1: GND -> /BM1397-1/GND1
- C84 pad 2: GND -> /BM1397-3/VDD3
- C85 pad 2: GND -> /BM1397-3/VDD3
- C86 pad 2: GND -> /BM1397-3/VDD3
- C87 pad 1: GND -> /BM1397-1/GND1
- C88 pad 1: GND -> /BM1397-1/GND1
- C88 pad 2: GND -> /BM1397-3/VDD3
- C90 pad 2: GND -> /BM1397-3/VDD3
- C91 pad 2: GND -> /BM1397-3/VDD3
- C93 pad 2: GND -> /BM1397-3/VDD3
- C94 pad 1: GND -> /BM1397-3/VDD3
- C96 pad 2: GND -> /BM1397-3/VDD3
- C97 pad 2: GND -> /BM1397-3/VDD3
- C99 pad 1: GND -> /BM1397-1/GND1
- C99 pad 2: GND -> /BM1397-3/VDD3
- D1 pad 1: /ESP32/5V -> /5V
- IC1 pad 13: GND -> /BM1397-1/GND1
- IC1 pad 19: GND -> /BM1397-1/GND1
- IC1 pad 21: unconnected-(IC1-TEMP_N-Pad21) -> /TEMP1_N
- IC1 pad 22: unconnected-(IC1-TEMP_P-Pad22) -> /TEMP1_P
- IC1 pad 34: GND -> /BM1397-1/GND1
- IC2 pad 13: GND -> /BM1397-1/GND1
- IC2 pad 19: GND -> /BM1397-1/GND1
- IC2 pad 34: GND -> /BM1397-1/GND1
- IC3 pad 13: GND -> /BM1397-3/VDD3
- IC3 pad 19: GND -> /BM1397-3/VDD3
- IC3 pad 20: Net-(IC3-PIN_MODE) -> /BM1397-3/VDD3
- IC3 pad 21: /TEMP1_N -> /TEMP2_N
- IC3 pad 22: /TEMP1_P -> /TEMP2_P
- IC3 pad 33: GND -> /BM1397-1/GND1
- IC3 pad 34: GND -> /BM1397-3/VDD3
- IC4 pad 13: GND -> /BM1397-3/VDD3
- IC4 pad 19: GND -> /BM1397-3/VDD3
- IC4 pad 20: Net-(IC4-PIN_MODE) -> /BM1397-3/VDD3
- IC4 pad 21: /TEMP2_N -> unconnected-(IC4-TEMP_N-Pad21)
- IC4 pad 22: /TEMP2_P -> unconnected-(IC4-TEMP_P-Pad22)
- IC4 pad 33: GND -> /BM1397-1/GND1
- IC4 pad 34: GND -> /BM1397-3/VDD3
- IC5 pad 21: unconnected-(IC5-TEMP_N-Pad21) -> /TEMP3_N
- IC5 pad 22: unconnected-(IC5-TEMP_P-Pad22) -> /TEMP3_P
- IC5 pad 33: GND -> /BM1397-3/VDD3
- IC6 pad 33: GND -> /BM1397-3/VDD3
- J4 pad 2: /ESP32/3V3 -> /3V3
- J5 pad 2: /ESP32/3V3 -> /3V3
- R13 pad 1: /ESP32/3V3 -> /3V3
- R14 pad 2: /ESP32/3V3 -> /3V3
- R15 pad 2: /ESP32/3V3 -> /3V3
- R16 pad 1: GND -> /BM1397-1/GND1
- R17 pad 1: GND -> /BM1397-1/GND1
- R18 pad 1: GND -> /BM1397-1/GND1
- R19 pad 2: GND -> /BM1397-1/GND1
- R20 pad 2: GND -> /BM1397-1/GND1
- R21 pad 1: GND -> /BM1397-1/GND1
- R22 pad 1: GND -> /BM1397-1/GND1
- R23 pad 1: GND -> /BM1397-1/GND1
- R32 pad 1: GND -> /BM1397-3/VDD3
- R33 pad 1: GND -> /BM1397-3/VDD3
- R34 pad 1: GND -> /BM1397-3/VDD3
- R35 pad 1: GND -> /BM1397-1/GND1
- R35 pad 2: GND -> /BM1397-3/VDD3
- R36 pad 1: GND -> /BM1397-1/GND1
- R36 pad 2: GND -> /BM1397-3/VDD3
- R37 pad 1: GND -> /BM1397-3/VDD3
- R38 pad 1: GND -> /BM1397-3/VDD3
- R39 pad 1: GND -> /BM1397-3/VDD3
- TP1 pad 1: /ESP32/3V3 -> /3V3
- U11 pad 2: GND -> /BM1397-3/VDD3
- U12 pad 2: GND -> /BM1397-3/VDD3
- U6 pad 2: /ESP32/3V3 -> /3V3
- U7 pad 2: GND -> /BM1397-1/GND1
- U8 pad 2: GND -> /BM1397-1/GND1
- X1 pad 2: GND -> /BM1397-1/GND1
Routing:
- added copper zone on B.Cu, net /BM1397-1/GND1
- added copper zone on F.Cu, net /BM1397-1/GND1
- added copper zone on B.Cu, net /BM1397-3/VDD3
- added copper zone on F.Cu, net /BM1397-3/VDD3
- added copper zone on F.Cu, net GND
