File: bitaxe_RGZ_204_MOD_C.kicad_pcb (KiCad board)
At the start: 4 copper layers, 56.5 x 99.8 mm, 137 parts, among them J1 54-00164, J2 Conn_01x02, J3 Conn_01x05, J4 Conn_01x04, J5 TC2030-IDC, J7 Conn_01x02, J8 USB_C_Receptacle_USB2.0, J9 Conn_01x04, Q1 CSD17311Q5, Q2 CSD17311Q5, Q4 2N7002K, SW1 GT-TC029B-H025-L1N, SW2 GT-TC029B-H025-L1N, U1 25MHz, U10 DS4432U+, U11 RT9080-33GJ5, U12 ESP32-S3-WROOM-1, U14 BM1366_mode1, U2 TXB0104RGYR, U5 MCP1824T-1802E, U6 MCP1824T-0802E, U7 EMC2101, U8 INA260, U9 TPS40305, Y1 32.768kHz

Commit message: no message
Parts:
- removed R11: 100k, Resistor_SMD:R_0402_1005Metric
- added C26: 0.1uF, Capacitor_SMD:C_0402_1005Metric, F.Cu at (110.8, 58.0)
- added Q3: S8050, Package_TO_SOT_SMD:SOT-23-3, F.Cu at (123.9, 55.0)
- added R17: 1k, Resistor_SMD:R_0402_1005Metric, F.Cu at (120.7, 56.3)
- added R18: 10k, Resistor_SMD:R_0402_1005Metric, F.Cu at (120.7, 54.8)
- added R19: 10, Resistor_SMD:R_0402_1005Metric, F.Cu at (120.7, 53.3)
- added U4: 176x320_st7789, bitaxe:ST7789-176x320, B.Cu at (114.2, 57.3)
- C22, C23: value 0.1uF -> 1uF
- J9: footprint Connector_PinSocket_2.54mm:PinSocket_1x04_P2.54mm_Vertical_SMD_Pin1Right -> Connector_PinSocket_2.54mm:PinSocket_1x04_P2.54mm_Vertical
- moved G*** 12.4 mm to (92.8, 87.9)
- moved R1 8.39 mm to (126.8, 110.1)
- moved R3 8.39 mm to (126.9, 94.4)
- moved R5 8.39 mm to (127.3, 107.3)
- moved SW1 8.39 mm to (130.2, 112.8)
- moved SW2 8.39 mm to (130.1, 121.5)
- moved J8 8.39 mm to (130.0, 100.8)
- moved FID2 7.35 mm to (130.3, 55.7)
- moved FID5 7.34 mm to (130.3, 55.7)
- moved TP18 6.25 mm to (131.4, 65.4)
- moved R8 6.25 mm to (110.9, 76.0), turned to 0 degrees
- moved C51 6.01 mm to (128.2, 89.1)
- moved C52 5.84 mm to (128.3, 90.6)
- moved C21 5.59 mm to (121.4, 106.7)
- moved U10 5.43 mm to (89.0, 103.2)
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Connections:
- U12 pad 12: unconnected-(U12-GPIO8/TOUCH8/ADC1_CH7/SUBSPICS1-Pad12) -> /ESP32/TFT_DC
- U12 pad 17: unconnected-(U12-GPIO9/TOUCH9/ADC1_CH8/FSPIHD/SUBSPIHD-Pad17) -> /ESP32/TFT_BLK
- U12 pad 4: unconnected-(U12-GPIO4/TOUCH4/ADC1_CH3-Pad4) -> /ESP32/TFT_RES
- U12 pad 5: unconnected-(U12-GPIO5/TOUCH5/ADC1_CH4-Pad5) -> /ESP32/TFT_SDA
- U12 pad 6: unconnected-(U12-GPIO6/TOUCH6/ADC1_CH5-Pad6) -> /ESP32/TFT_SCL
- U12 pad 7: unconnected-(U12-GPIO7/TOUCH7/ADC1_CH6-Pad7) -> /ESP32/TFT_CS
Routing:
- net /ESP32/TFT_RES: track 0.00 -> 36.9 mm, vias 0 -> 2
- net /ESP32/TFT_DC: track 0.00 -> 35.6 mm, vias 0 -> 2
- net /ESP32/TFT_SDA: track 0.00 -> 35.6 mm, vias 0 -> 2
- net /ESP32/TFT_SCL: track 0.00 -> 34.5 mm, vias 0 -> 2
- net /ESP32/TFT_CS: track 0.00 -> 33.2 mm, vias 0 -> 2
- net /ESP32/TFT_BLK: track 0.00 -> 32.6 mm, vias 0 -> 3
- net /TX: track 40.4 -> 17.9 mm
- net /SDA: track 128.7 -> 143.0 mm
- net GND: track 147.4 -> 160.2 mm, vias 83 -> 85
- net Net-(U4-LEDK): track 0.00 -> 11.8 mm, vias 0 -> 1
- net /ESP32/EN: track 81.0 -> 71.6 mm
- net /Power/SW: track 5.41 -> 13.6 mm
- net /RX: track 25.7 -> 18.0 mm
- net Net-(Q1-G): track 11.9 -> 17.1 mm
- net Net-(U9-BP): track 16.8 -> 12.0 mm
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- added copper zone on B.Cu, net (none)
- added copper zone on F.Cu, net (none)
Other:
- outline, holes or cut-outs redrawn
- board text added: "204_MOD"
- board text removed: "204"
