File: bitaxe_RGZ_204_MOD_C.kicad_sch (KiCad schematic)
At the start: 16 parts, among them J1 54-00164

Commit message: no message
Parts:
- J1: PARTNO 54-00164 -> 54-00164 C319134
Changed lines of the file:
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@@
     )
     (instances
-      (project "bitaxeUltra"
+      (project "bitaxe_RGZ_204_MOD_C"
         (path "/e63e39d7-6ac0-4ffd-8aa3-1841a4541b55"
           (reference "FID2") (unit 1)
@@
     )
     (instances
-      (project "bitaxeUltra"
+      (project "bitaxe_RGZ_204_MOD_C"
         (path "/e63e39d7-6ac0-4ffd-8aa3-1841a4541b55"
           (reference "FID3") (unit 1)
@@
     )
     (instances
-      (project "bitaxeUltra"
+      (project "bitaxe_RGZ_204_MOD_C"
         (path "/e63e39d7-6ac0-4ffd-8aa3-1841a4541b55"
           (reference "FID4") (unit 1)
@@
     )
     (instances
-      (project "bitaxeUltra"
+      (project "bitaxe_RGZ_204_MOD_C"
         (path "/e63e39d7-6ac0-4ffd-8aa3-1841a4541b55"
           (reference "FID6") (unit 1)
@@
       (effects (font (size 1.27 1.27)) hide)
     )
-    (property "PARTNO" "54-00164" (at 64.77 45.72 0)
+    (property "PARTNO" "54-00164  C319134 " (at 64.77 45.72 0)
       (effects (font (size 1.27 1.27)) hide)
     )
@@
     (pin "3")
     (instances
-      (project "bitaxeUltra"
+      (project "bitaxe_RGZ_204_MOD_C"
         (path "/e63e39d7-6ac0-4ffd-8aa3-1841a4541b55"
           (reference "J1") (unit 1)
@@
     (pin "1")
     (instances
-      (project "bitaxeUltra"
+      (project "bitaxe_RGZ_204_MOD_C"
         (path "/e63e39d7-6ac0-4ffd-8aa3-1841a4541b55"
           (reference "H7") (unit 1)
@@
     )
     (instances
-      (project "bitaxeUltra"
+      (project "bitaxe_RGZ_204_MOD_C"
         (path "/e63e39d7-6ac0-4ffd-8aa3-1841a4541b55"
           (reference "FID1") (unit 1)
@@
     )
     (instances
-      (project "bitaxeUltra"
+      (project "bitaxe_RGZ_204_MOD_C"
         (path "/e63e39d7-6ac0-4ffd-8aa3-1841a4541b55"
           (reference "FID8") (unit 1)
@@
     )
     (instances
-      (project "bitaxeUltra"
+      (project "bitaxe_RGZ_204_MOD_C"
         (path "/e63e39d7-6ac0-4ffd-8aa3-1841a4541b55"
           (reference "FID5") (unit 1)
@@
     )
     (instances
-      (project "bitaxeUltra"
+      (project "bitaxe_RGZ_204_MOD_C"
         (path "/e63e39d7-6ac0-4ffd-8aa3-1841a4541b55"
           (reference "H6") (unit 1)
@@
     )
     (instances
-      (project "bitaxeUltra"
+      (project "bitaxe_RGZ_204_MOD_C"
         (path "/e63e39d7-6ac0-4ffd-8aa3-1841a4541b55"
           (reference "FID7") (unit 1)
@@
     )
     (instances
-      (project "bitaxeUltra"
+      (project "bitaxe_RGZ_204_MOD_C"
         (path "/e63e39d7-6ac0-4ffd-8aa3-1841a4541b55"
           (reference "H5") (unit 1)
@@
     (pin "1")
     (instances
-      (project "bitaxeUltra"
+      (project "bitaxe_RGZ_204_MOD_C"
         (path "/e63e39d7-6ac0-4ffd-8aa3-1841a4541b55"
           (reference "H9") (unit 1)
@@
     (pin "1")
     (instances
-      (project "bitaxeUltra"
+      (project "bitaxe_RGZ_204_MOD_C"
         (path "/e63e39d7-6ac0-4ffd-8aa3-1841a4541b55"
           (reference "H8") (unit 1)
@@
     (pin "1")
     (instances
-      (project "bitaxeUltra"
+      (project "bitaxe_RGZ_204_MOD_C"
         (path "/e63e39d7-6ac0-4ffd-8aa3-1841a4541b55"
           (reference "H10") (unit 1)
@@
     )
     (instances
-      (project "bitaxeUltra"
+      (project "bitaxe_RGZ_204_MOD_C"
         (path "/e63e39d7-6ac0-4ffd-8aa3-1841a4541b55"
           (reference "#G1") (unit 1)
@@
     )
     (instances
-      (project "bitaxeUltra"
+      (project "bitaxe_RGZ_204_MOD_C"
         (path "/e63e39d7-6ac0-4ffd-8aa3-1841a4541b55"
           (reference "U3") (unit 1)
@@
     )
     (instances
-      (project "bitaxeUltra"
+      (project "bitaxe_RGZ_204_MOD_C"
         (path "/e63e39d7-6ac0-4ffd-8aa3-1841a4541b55" (page "4"))
       )
@@
     )
     (instances
-      (project "bitaxeUltra"
+      (project "bitaxe_RGZ_204_MOD_C"
         (path "/e63e39d7-6ac0-4ffd-8aa3-1841a4541b55" (page "5"))
       )
@@
     )
     (instances
-      (project "bitaxeUltra"
+      (project "bitaxe_RGZ_204_MOD_C"
         (path "/e63e39d7-6ac0-4ffd-8aa3-1841a4541b55" (page "2"))
       )
@@
     )
     (instances
-      (project "bitaxeUltra"
+      (project "bitaxe_RGZ_204_MOD_C"
         (path "/e63e39d7-6ac0-4ffd-8aa3-1841a4541b55" (page "3"))
       )
