File: NerdAxe_ultra.kicad_pcb (KiCad board)
At the start: 4 copper layers, 56.5 x 99.8 mm, 110 parts, among them J3 Conn_01x05, J4 Conn_01x04, J7 Conn_01x02, Q1 CSD17311Q5, Q2 CSD17311Q5, U1 25MHz, U10 DS4432U+, U14 BM1366_mode0, U2 TXB0104RGYR, U3 T-Display-S3, U5 MCP1824T-1802E, U6 MCP1824T-0802E, U7 EMC2101, U8 INA260, U9 TPS40305

Commit message: Manufacturing files
Parts:
- added G***: LOGO, bitaxe:nerdaxeLogo2, B.Cu at (48.0, 80.3)
Other:
- board text added: "NerdAxeUltra"

Commit message: NerdAxe update v1.1
Parts:
- removed C32: 470pF, Capacitor_SMD:C_0402_1005Metric
- removed DC1: DC-044K-D025, lcsc:DC-IN-TH_DC-044K-D025
- removed the G*** at (48.0, 80.3)
- removed the G*** at (127.4, 101.4)
- removed J3: Conn_01x05, Connector_PinHeader_2.54mm:PinHeader_1x05_P2.54mm_Vertical
- removed J7: Conn_01x02, Connector_PinHeader_2.54mm:PinHeader_1x02_P2.54mm_Vertical
- removed R11: 100k, Resistor_SMD:R_0402_1005Metric
- removed R7, R8: 100, Resistor_SMD:R_0402_1005Metric
- removed TP20, TP37, TP39, TP5, TP6: TestPoint, TestPoint:TestPoint_Pad_D1.5mm
- removed kibuzzard-63D74789: G***, kibuzzard-63D74789
- added D1: US1D, Diode_SMD:D_SMA, F.Cu at (114.3, 77.8)
- added FID1: Fiducial, Fiducial:Fiducial_1mm_Mask2mm, F.Cu at (78.5, 57.8)
- added FID2: Fiducial, Fiducial:Fiducial_1mm_Mask2mm, F.Cu at (125.6, 51.1)
- added FID3: Fiducial, Fiducial:Fiducial_1mm_Mask2mm, F.Cu at (77.9, 138.2)
- added FID4: Fiducial, Fiducial:Fiducial_1mm_Mask2mm, F.Cu at (132.6, 137.8)
- added FID5: Fiducial, Fiducial:Fiducial_1mm_Mask2mm, B.Cu at (125.6, 51.1)
- added FID6: Fiducial, Fiducial:Fiducial_1mm_Mask2mm, B.Cu at (132.6, 137.8)
- added FID7: Fiducial, Fiducial:Fiducial_1mm_Mask2mm, B.Cu at (78.5, 57.8)
- added FID8: Fiducial, Fiducial:Fiducial_1mm_Mask2mm, B.Cu at (77.9, 138.2)
- added G***: LOGO, bitaxe:nerdAxeLogo6, B.Cu at (95.9, 83.9)
- added J1: 54-00164, bitaxe:BarrelJack_Wuerth_694106106102_2.0x5.5mm, B.Cu at (127.9, 83.5)
- added Q3: 2N7002K, Package_TO_SOT_SMD:SOT-323_SC-70, F.Cu at (107.6, 81.2)
- added R1: 10k, Resistor_SMD:R_0402_1005Metric, F.Cu at (120.4, 112.0)
- added R5: 1M, Resistor_SMD:R_0402_1005Metric, F.Cu at (122.6, 90.6)
- added R6: 10k, Resistor_SMD:R_0402_1005Metric, F.Cu at (107.4, 77.1)
- H1, H2, H3, H4: footprint MountingHole:MountingHole_2.2mm_M2 -> MountingHole:MountingHole_3mm_Pad_Via
- moved H1 93.3 mm to (78.5, 51.1)
- moved H4 93.2 mm to (78.5, 143.8)
- moved TP11 34.5 mm to (119.9, 121.9)
- moved TP12 33.5 mm to (115.8, 119.1)
- moved R16 31.3 mm to (86.4, 74.8)
- moved R9 28.4 mm to (100.6, 111.4)
- moved U7 28.0 mm to (100.8, 115.8)
- moved C33 27.0 mm to (101.7, 111.4)
- moved C44 26.6 mm to (84.2, 74.8)
- moved TP4 25.2 mm to (119.9, 115.2), turned to 0 degrees
- moved U10 25.0 mm to (85.6, 78.6), turned to 90 degrees
- moved R17 23.9 mm to (86.1, 82.4)
- moved TP3 23.7 mm to (122.4, 117.9)
- moved TP2 22.3 mm to (119.9, 119.4)
- moved TP15 20.0 mm to (103.9, 137.8)
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Connections:
- net /TEMP_N renamed /BM1366/ADDR1
- net /TEMP_P renamed /BM1366/ADDR0
- C16 pad 1: /BM1366/MODE_1 -> /BM1366/0V8
- C16 pad 2: /BM1366/0V8 -> GND
- C18 pad 2: /BM1366/VDD4_1 -> GND
- C2 pad 1: /BM1366/VDD4_0 -> GND
- C4 pad 1: /BM1366/MODE_OUT -> GND
- TP46 pad 1: /BM1366/MODE_0 -> /BM1366/INV_CL0
- TP47 pad 1: /BM1366/MODE_1 -> /BM1366/PIN_MODE
- U14 pad 12: /BM1366/MODE_OUT -> GND
- U14 pad 17: /BM1366/MODE_1 -> GND
- U14 pad 18: /BM1366/MODE_0 -> /BM1366/PIN_MODE
- U14 pad 19: /BM1366/NC -> /BM1366/INV_CL0
- U14 pad 25: /BM1366/VDD4_1 -> GND
- U14 pad 4: /BM1366/VDD4_0 -> GND
- U3 pad 12: /5V -> Net-(D1-K)
- U3 pad 13: /3V3 -> /TTGO/3V
- U3 pad 5: unconnected-(U3-GPIO10-Pad5) -> /Power/PWR_EN
- U3 pad 7: unconnected-(U3-GPIO12-Pad7) -> /PLUG_SENSE
- U7 pad 2: Net-(U7-DP) -> unconnected-(U7-DP-Pad2)
- U7 pad 3: Net-(U7-DN) -> unconnected-(U7-DN-Pad3)
Routing:
- net /3V3: track 102.8 -> 24.0 mm, vias 9 -> 7
- net /BM1366/ADDR1: track 72.2 -> 9.05 mm
- net /BM1366/ADDR0: track 73.5 -> 13.8 mm
- net /PLUG_SENSE: track 0.00 -> 40.7 mm, vias 0 -> 2
- net /BM1366/RST_N: track 62.2 -> 28.6 mm
- net /Fan/FAN_TACH: track 22.3 -> 54.1 mm
- net /BM1366/CI: track 65.3 -> 33.9 mm
- net /BM1366/RO: track 66.2 -> 35.8 mm
- net /Power/PWR_EN: track 0.00 -> 26.4 mm, vias 0 -> 1
- net GND: track 74.7 -> 101.0 mm, vias 48 -> 57
- net /Fan/FAN_PWM: track 32.2 -> 58.5 mm, vias 0 -> 2
- net /BM1366/NC: track 24.0 -> 0.00 mm, vias 1 -> 0
- net /BM1366/1V8: track 114.6 -> 90.6 mm
- net /BM1366/MODE_1: track 23.7 -> 0.00 mm, vias 1 -> 0
- net /Power/OUT0: track 43.9 -> 20.8 mm, vias 2 -> 0
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- added copper zone on B.Cu, net /5V
- added copper zone on In2.Cu, net /5V
- added copper zone on B.Cu, net /VIN
Other:
- board size 56.5 x 99.8 mm -> 61.1 x 99.8 mm
- board text added: "5V/4A"
- board text added: "BM1366 NERDAXE V1.0.1"
- board text removed: "1V8"
- board text removed: "5V Power 3A"
- board text removed: "BM1366 NERDAXE V1"
- board text removed: "NerdAxeUltra"
- board text removed: "RST"
- board text removed: "RXI"
- board text removed: "TXO"
- board text removed: "VERIFY POLARITY"
