File: NerdAxe_ultra.kicad_sch (KiCad schematic)
At the start: 7 parts

Commit message: Manufacturing files
Other:
- note added: "NerdAxe_ultra"
- note removed: "bitaxe, TTGO"
Changed lines of the file:
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@@
     (stroke (width 0) (type default))
   )
-  (text "bitaxe, TTGO" (at 160.655 186.055 0)
+  (text "NerdAxe_ultra" (at 160.655 186.055 0)
     (effects (font (size 5 5) (thickness 1) bold) (justify left bottom))
   )
@@
     )
     (instances
-      (project "bitaxeTTGO"
+      (project "NerdAxe_ultra"
         (path "/e63e39d7-6ac0-4ffd-8aa3-1841a4541b55"
           (reference "H3") (unit 1)
@@
     )
     (instances
-      (project "bitaxeTTGO"
+      (project "NerdAxe_ultra"
         (path "/e63e39d7-6ac0-4ffd-8aa3-1841a4541b55"
           (reference "H2") (unit 1)
@@
     )
     (instances
-      (project "bitaxeTTGO"
+      (project "NerdAxe_ultra"
         (path "/e63e39d7-6ac0-4ffd-8aa3-1841a4541b55"
           (reference "H1") (unit 1)
@@
     )
     (instances
-      (project "bitaxeTTGO"
+      (project "NerdAxe_ultra"
         (path "/e63e39d7-6ac0-4ffd-8aa3-1841a4541b55"
           (reference "H6") (unit 1)
@@
     )
     (instances
-      (project "bitaxeTTGO"
+      (project "NerdAxe_ultra"
         (path "/e63e39d7-6ac0-4ffd-8aa3-1841a4541b55"
           (reference "H5") (unit 1)
@@
         )
       )
-      (project "bitaxeTTGO"
+      (project "NerdAxe_ultra"
         (path "/e63e39d7-6ac0-4ffd-8aa3-1841a4541b55"
           (reference "DC1") (unit 1)
@@
     )
     (instances
-      (project "bitaxeTTGO"
+      (project "NerdAxe_ultra"
         (path "/e63e39d7-6ac0-4ffd-8aa3-1841a4541b55"
           (reference "H4") (unit 1)
@@
     )
     (instances
-      (project "bitaxeTTGO"
+      (project "NerdAxe_ultra"
         (path "/e63e39d7-6ac0-4ffd-8aa3-1841a4541b55" (page "6"))
       )
@@
     )
     (instances
-      (project "bitaxeTTGO"
+      (project "NerdAxe_ultra"
         (path "/e63e39d7-6ac0-4ffd-8aa3-1841a4541b55" (page "4"))
       )
@@
     )
     (instances
-      (project "bitaxeTTGO"
+      (project "NerdAxe_ultra"
         (path "/e63e39d7-6ac0-4ffd-8aa3-1841a4541b55" (page "5"))
       )
@@
     )
     (instances
-      (project "bitaxeTTGO"
+      (project "NerdAxe_ultra"
         (path "/e63e39d7-6ac0-4ffd-8aa3-1841a4541b55" (page "2"))
       )

Commit message: NerdAxe update v1.1
Parts:
- removed DC1: DC-044K-D025, lcsc:DC-IN-TH_DC-044K-D025, symbol lcsc:DC-044K-D025
- added FID1, FID2, FID3, FID4, FID5, FID6, FID7, FID8: Fiducial, Fiducial:Fiducial_1mm_Mask2mm, symbol Mechanical:Fiducial
- added J1: 54-00164, bitaxe:BarrelJack_Wuerth_694106106102_2.0x5.5mm, symbol Connector:Barrel_Jack_Switch
- H1, H2, H3, H4: footprint MountingHole:MountingHole_2.2mm_M2 -> MountingHole:MountingHole_3mm_Pad_Via; symbol Mechanical:MountingHole -> Mechanical:MountingHole_Pad; now in the parts list
Connections:
- net GND: now also H1.1, H2.1, H3.1, H4.1, J1.2
- net VIN: now also J1.1
- new net PLUG_SENSE: J1.3
Other:
- sheet BM1366 ports: added none; removed TEMP_N, TEMP_P
- sheet Fan ports: added none; removed TEMP_N, TEMP_P
- sheet Power ports: added PWR_EN; removed none
- sheet TTGO ports: added 3V3, PLUG_SENSE, PWR_EN; removed 3V

Commit message: minimal changes
Other:
- note added: "NerdAxe"
- note added: "credits to Bitaxe project members"
- note removed: "NerdAxe_ultra"
- title: le bitaxeTTGO -> bitaxeTTGO
Changed lines of the file:
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@@
   (paper "A")
   (title_block
-    (title "le bitaxeTTGO")
+    (title "bitaxeTTGO")
     (date "2023-07-10")
     (rev "0")
@@
     (stroke (width 0) (type default))
   )
-  (text "NerdAxe_ultra" (at 160.655 186.055 0)
+  (text "credits to Bitaxe project members" (at 161.925 185.42 0)
+    (effects (font (size 3 3) (thickness 1) bold) (justify left bottom))
+  )
+  (text "NerdAxe" (at 161.29 180.34 0)
     (effects (font (size 5 5) (thickness 1) bold) (justify left bottom))
   )
