File: TTGO.kicad_sch (KiCad schematic)
At the start: 1 part, among them U3 T-Display-S3

Commit message: NerdAxe update v1.1
Parts:
- added D1: US1D, Diode_SMD:D_SMA, symbol Diode:US1D
- added R20: 1M, Resistor_SMD:R_0402_1005Metric, symbol Device:R_US
- added R20: 10k, Resistor_SMD:R_0402_1005Metric, symbol Device:R_US
Connections:
- net 3V: no longer U3.1 (3V)
- net 5V: now also D1.2 (A); no longer U3.12 (5V)
- net PWR_EN: now reaches U3.5 (GPIO10)
- net PWR_EN: now also R20.2
- net PLUG_SENSE: now reaches U3.7 (GPIO12)
- net PLUG_SENSE: now also R20.2
- new net: D1.1 (K), U3.12 (5V)
- new net 3V3: R20.1, R20.1, U3.1 (3V)
Changed lines of the file:
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@@
 (kicad_sch (version 20230121) (generator eeschema)
   (paper "A4")
-  (wire (pts (xy 104.14 96.52) (xy 109.855 96.52))
+  (junction (at 72.39 83.82) (diameter 0) (color 0 0 0 0)
+  )
+  (junction (at 72.39 66.04) (diameter 0) (color 0 0 0 0)
+  )
+  (junction (at 87.63 78.74) (diameter 0) (color 0 0 0 0)
+  )
+  (wire (pts (xy 108.585 98.425) (xy 108.585 96.52))
+    (stroke (width 0) (type default))
+  )
+  (wire (pts (xy 105.41 98.425) (xy 108.585 98.425))
+    (stroke (width 0) (type default))
+  )
+  (wire (pts (xy 95.25 98.425) (xy 97.79 98.425))
+    (stroke (width 0) (type default))
+  )
+  (wire (pts (xy 87.63 76.2) (xy 87.63 78.74))
+    (stroke (width 0) (type default))
+  )
+  (wire (pts (xy 72.39 77.47) (xy 72.39 83.82))
+    (stroke (width 0) (type default))
+  )
+  (wire (pts (xy 72.39 66.04) (xy 72.39 69.85))
+    (stroke (width 0) (type default))
+  )
+  (wire (pts (xy 69.85 83.82) (xy 72.39 83.82))
+    (stroke (width 0) (type default))
+  )
+  (wire (pts (xy 72.39 66.04) (xy 87.63 66.04))
     (stroke (width 0) (type default))
   )
@@
     (stroke (width 0) (type default))
   )
+  (wire (pts (xy 85.725 78.74) (xy 87.63 78.74))
+    (stroke (width 0) (type default))
+  )
   (wire (pts (xy 132.715 91.44) (xy 138.43 91.44))
     (stroke (width 0) (type default))
@@
     (stroke (width 0) (type default))
   )
+  (wire (pts (xy 87.63 78.74) (xy 109.855 78.74))
+    (stroke (width 0) (type default))
+  )
   (wire (pts (xy 109.855 93.98) (xy 104.14 93.98))
     (stroke (width 0) (type default))
@@
     (stroke (width 0) (type default))
   )
+  (wire (pts (xy 69.215 66.04) (xy 72.39 66.04))
+    (stroke (width 0) (type default))
+  )
   (wire (pts (xy 132.715 93.98) (xy 138.43 93.98))
+    (stroke (width 0) (type default))
+  )
+  (wire (pts (xy 108.585 96.52) (xy 109.855 96.52))
+    (stroke (width 0) (type default))
+  )
+  (wire (pts (xy 87.63 68.58) (xy 87.63 66.04))
+    (stroke (width 0) (type default))
+  )
+  (wire (pts (xy 72.39 83.82) (xy 109.855 83.82))
     (stroke (width 0) (type default))
   )
@@
     (effects (font (size 1.27 1.27)) (justify left bottom))
   )
+  (label "3V3" (at 78.74 66.04 0) (fields_autoplaced)
+    (effects (font (size 1.27 1.27)) (justify left bottom))
+  )
   (label "GND" (at 138.43 68.58 180) (fields_autoplaced)
     (effects (font (size 1.27 1.27)) (justify right bottom))
@@
     (effects (font (size 1.27 1.27)) (justify right bottom))
   )
-  (label "3V" (at 104.14 68.58 0) (fields_autoplaced)
+  (label "3V3" (at 104.14 68.58 0) (fields_autoplaced)
     (effects (font (size 1.27 1.27)) (justify left bottom))
   )
@@
     )
   )
-  (hierarchical_label "5V" (shape input) (at 104.14 96.52 180) (fields_autoplaced)
+  (hierarchical_label "5V" (shape input) (at 95.25 98.425 180) (fields_autoplaced)
     (effects (font (size 1.27 1.27)) (justify right))
   )
@@
     (effects (font (size 1.27 1.27)) (justify left))
   )
+  (hierarchical_label "PLUG_SENSE" (shape input) (at 69.85 83.82 180) (fields_autoplaced)
+    (effects (font (size 1.27 1.27)) (justify right))
+  )
   (hierarchical_label "3V" (shape input) (at 144.145 96.52 0) (fields_autoplaced)
     (effects (font (size 1.27 1.27)) (justify left))
@@
     (effects (font (size 1.27 1.27)) (justify right))
   )
+  (hierarchical_label "3V3" (shape input) (at 69.215 66.04 180) (fields_autoplaced)
+    (effects (font (size 1.27 1.27)) (justify right))
+  )
+  (hierarchical_label "PWR_EN" (shape output) (at 85.725 78.74 180) (fields_autoplaced)
+    (effects (font (size 1.27 1.27)) (justify right))
+  )
   (hierarchical_label "RX" (shape input) (at 144.145 78.74 0) (fields_autoplaced)
     (effects (font (size 1.27 1.27)) (justify left))
+  )
+  (symbol (lib_id "Diode:US1D") (at 101.6 98.425 180) (unit 1)
+    (in_bom yes) (on_board yes) (dnp no)
+    (property "Reference" "D1" (at 97.79 100.33 0)
+      (effects (font (size 1.27 1.27)))
+    )
+    (property "Value" "US1D" (at 105.41 100.33 0)
+      (effects (font (size 1.27 1.27)))
+    )
+    (property "Footprint" "Diode_SMD:D_SMA" (at 101.6 93.98 0)
+      (effects (font (size 1.27 1.27)) hide)
+    )
+    (property "Datasheet" "https://www.diodes.com/assets/Datasheets/ds16008.pdf" (at 101.6 98.425 0)
+      (effects (font (size 1.27 1.27)) hide)
+    )
+    (property "Sim.Device" "D" (at 101.6 98.425 0)
+      (effects (font (size 1.27 1.27)) hide)
+    )
+    (property "Sim.Pins" "1=K 2=A" (at 101.6 98.425 0)
+      (effects (font (size 1.27 1.27)) hide)
+    )
+    (pin "1")
+    (pin "2")
+    (instances
+      (project "NerdAxe_ultra"
+        (path "/e63e39d7-6ac0-4ffd-8aa3-1841a4541b55/26d98239-cc99-433b-80b9-07c779389fec"
+          (reference "D1") (unit 1)
+        )
+      )
+    )
   )
   (symbol (lib_id "bitaxe:T-Display-S3") (at 135.255 63.5 0) (unit 1)
@@
         )
       )
+    )
+  )
+  (symbol (lib_id "Device:R_US") (at 72.39 73.66 0) (unit 1)
+    (in_bom yes) (on_board yes) (dnp no) (fields_autoplaced)
+    (property "Reference" "R20" (at 74.295 72.39 0)
+      (effects (font (size 1.27 1.27)) (justify left))
+    )
+    (property "Value" "1M" (at 74.295 74.93 0)
+      (effects (font (size 1.27 1.27)) (justify left))
+    )
+    (property "Footprint" "Resistor_SMD:R_0402_1005Metric" (at 73.406 73.914 90)
+      (effects (font (size 1.27 1.27)) hide)
+    )
+    (property "Datasheet" "~" (at 72.39 73.66 0)
+      (effects (font (size 1.27 1.27)) hide)
+    )
+    (property "DK" "311-1.00MLRCT-ND" (at 72.39 73.66 0)
+      (effects (font (size 1.27 1.27)) hide)
+    )
+    (property "PARTNO" "RC0402FR-071ML" (at 72.39 73.66 0)
+      (effects (font (size 1.27 1.27)) hide)
+    )
+    (pin "1")
+    (pin "2")
+    (instances
+      (project "esp32"
+        (path "/dcd2fc1c-da48-40a9-b97c-5712d9530f4f"
+          (reference "R20") (unit 1)
+        )
+      )
+      (project "NerdAxe_ultra"
+        (path "/e63e39d7-6ac0-4ffd-8aa3-1841a4541b55/26d98239-cc99-433b-80b9-07c779389fec"
+          (reference "R5") (unit 1)
+        )
+      )
+    )
+  )
+  (symbol (lib_id "Device:R_US") (at 87.63 72.39 0) (unit 1)
+    (in_bom yes) (on_board yes) (dnp no) (fields_autoplaced)
+    (property "Reference" "R20" (at 89.535 71.12 0)
+      (effects (font (size 1.27 1.27)) (justify left))
+    )
+    (property "Value" "10k" (at 89.535 73.66 0)
+      (effects (font (size 1.27 1.27)) (justify left))
+    )
+    (property "Footprint" "Resistor_SMD:R_0402_1005Metric" (at 88.646 72.644 90)
+      (effects (font (size 1.27 1.27)) hide)
+    )
+    (property "Datasheet" "~" (at 87.63 72.39 0)
+      (effects (font (size 1.27 1.27)) hide)
+    )
+    (property "DK" "311-10KJRCT-ND" (at 87.63 72.39 0)
+      (effects (font (size 1.27 1.27)) hide)
+    )
+    (property "PARTNO" "RC0402JR-0710KL" (at 87.63 72.39 0)
+      (effects (font (size 1.27 1.27)) hide)
+    )
+    (pin "1")
+    (pin "2")
+    (instances
+      (project "esp32"
+        (path "/dcd2fc1c-da48-40a9-b97c-5712d9530f4f"
+          (reference "R20") (unit 1)
+        )
+      )
+      (project "NerdAxe_ultra"
+        (path "/e63e39d7-6ac0-4ffd-8aa3-1841a4541b55/26d98239-cc99-433b-80b9-07c779389fec"
+          (reference "R6") (unit 1)
+        )
+      )

Commit message: minimal changes
Other:
- title: (none) -> NerdAxe
Changed lines of the file:
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@@
 (kicad_sch (version 20230121) (generator eeschema)
-  (paper "A4")
+  (paper "A")
+  (title_block
+    (title "NerdAxe")
+    (rev "1.1")
+  )
   (junction (at 72.39 83.82) (diameter 0) (color 0 0 0 0)
   )
